File: Hardware/Dreamcast_VGA_Adapter.sch (KiCad schematic (older format))
At the start: 38 parts, among them J1 AudioJack3, J2 DB15_Female_HighDensity_Mount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, J3 Conn_01x03, J4 Conn_01x06, J5 Conn_01x06, SW1 SW_DIP_x02, U1 THS7316, U2 74HCT2G34

Commit message: Update Dreamcast_VGA_Adapter.sch
Parts:
- added C8: 100uCP, Capacitor_THT:CP_Radial_D5.0mm_P2.00mm, symbol Device:CP
Connections:
- wire segments 129 -> 133
Changed lines of the file:
@@
 	0    1    1    0
 $EndComp
-Text Label 1650 6150 2    50   ~ 0
-5V
 Text Label 900  6150 0    50   ~ 0
 5V_IN
@@
 	-1   0    0    1
 $EndComp
+$Comp
+L Device:CP C8
+U 1 1 5F681767
+P 2200 6400
+F 0 "C8" H 2318 6446 50  0000 L CNN
+F 1 "100uCP" H 2318 6355 50  0000 L CNN
+F 2 "Capacitor_THT:CP_Radial_D5.0mm_P2.00mm" H 2238 6250 50  0001 C CNN
+F 3 "http://www.rubycon.co.jp/en/catalog/e_pdfs/aluminum/e_zlh.pdf" H 2200 6400 50  0001 C CNN
+F 4 "16ZLH100MEFC5X11" H 2200 6400 50  0001 C CNN "Manufacturer Part Number"
+	1    2200 6400
+	1    0    0    -1
+$EndComp
+Wire Wire Line
+	1650 6150 2200 6150
+Connection ~ 1650 6150
+Wire Wire Line
+	2200 6250 2200 6150
+Connection ~ 2200 6150
+Wire Wire Line
+	2200 6150 2700 6150
+Text Label 2700 6150 2    50   ~ 0
+5V
+Text Label 2200 6750 1    50   ~ 0
+GND
+Wire Wire Line
+	2200 6750 2200 6550
 $EndSCHEMATC

Commit message: Update Dreamcast_VGA_Adapter.sch
Parts:
- added R6, R7, R8: 75R, Resistor_SMD:R_0805_2012Metric_Pad1.15x1.40mm_HandSolder, symbol Device:R
Connections:
- wire segments 133 -> 142
Other:
- moved on the sheet: C12, C13, C14
Changed lines of the file:
@@
 	1    0    0    -1
 $EndComp
-Text Label 3900 1800 0    50   ~ 0
+Text Label 3350 1800 0    50   ~ 0
 DAC_GREEN
-Text Label 3900 2700 0    50   ~ 0
+Text Label 3350 2700 0    50   ~ 0
 DAC_BLUE
 Text Label 6100 3350 1    50   ~ 0
@@
 Wire Wire Line
 	5100 3100 5100 3250
-Text Label 3900 3600 0    50   ~ 0
+Text Label 3350 3600 0    50   ~ 0
 DAC_RED
-Wire Wire Line
-	3900 1800 4350 1800
-Wire Wire Line
-	3900 2700 4350 2700
-Wire Wire Line
-	3900 3600 4350 3600
 Wire Wire Line
 	6600 2700 6900 2700
@@
 L Device:C C12
 U 1 1 5F1E6679
-P 4350 2000
-F 0 "C12" H 4465 2046 50  0000 L CNN
-F 1 "10pC" H 4465 1955 50  0000 L CNN
-F 2 "Capacitor_SMD:C_0805_2012Metric_Pad1.15x1.40mm_HandSolder" H 4388 1850 50  0001 C CNN
-F 3 "~" H 4350 2000 50  0001 C CNN
-F 4 "DNP" H 4350 2000 50  0001 C CNN "Manufacturer Part Number"
-	1    4350 2000
+P 3950 2000
+F 0 "C12" H 4065 2046 50  0000 L CNN
+F 1 "10pC" H 4065 1955 50  0000 L CNN
+F 2 "Capacitor_SMD:C_0805_2012Metric_Pad1.15x1.40mm_HandSolder" H 3988 1850 50  0001 C CNN
+F 3 "~" H 3950 2000 50  0001 C CNN
+F 4 "DNP" H 3950 2000 50  0001 C CNN "Manufacturer Part Number"
+	1    3950 2000
 	1    0    0    -1
 $EndComp
@@
 L Device:C C13
 U 1 1 5F1E76F3
-P 4350 2900
-F 0 "C13" H 4465 2946 50  0000 L CNN
-F 1 "10pC" H 4465 2855 50  0000 L CNN
-F 2 "Capacitor_SMD:C_0805_2012Metric_Pad1.15x1.40mm_HandSolder" H 4388 2750 50  0001 C CNN
-F 3 "~" H 4350 2900 50  0001 C CNN
-F 4 "DNP" H 4350 2900 50  0001 C CNN "Manufacturer Part Number"
-	1    4350 2900
+P 3950 2900
+F 0 "C13" H 4065 2946 50  0000 L CNN
+F 1 "10pC" H 4065 2855 50  0000 L CNN
+F 2 "Capacitor_SMD:C_0805_2012Metric_Pad1.15x1.40mm_HandSolder" H 3988 2750 50  0001 C CNN
+F 3 "~" H 3950 2900 50  0001 C CNN
+F 4 "DNP" H 3950 2900 50  0001 C CNN "Manufacturer Part Number"
+	1    3950 2900
 	1    0    0    -1
 $EndComp
@@
 L Device:C C14
 U 1 1 5F1E806E
-P 4350 3800
-F 0 "C14" H 4465 3846 50  0000 L CNN
-F 1 "10pC" H 4465 3755 50  0000 L CNN
-F 2 "Capacitor_SMD:C_0805_2012Metric_Pad1.15x1.40mm_HandSolder" H 4388 3650 50  0001 C CNN
-F 3 "~" H 4350 3800 50  0001 C CNN
-F 4 "DNP" H 4350 3800 50  0001 C CNN "Manufacturer Part Number"
-	1    4350 3800
-	1    0    0    -1
-$EndComp
-Text Label 4350 2350 1    50   ~ 0
-GND
-Wire Wire Line
-	4350 2150 4350 2350
-Text Label 4350 3250 1    50   ~ 0
-GND
-Wire Wire Line
-	4350 3050 4350 3250
-Text Label 4350 4150 1    50   ~ 0
-GND
-Wire Wire Line
-	4350 3950 4350 4150
-Wire Wire Line
-	4350 3600 4350 3650
-Wire Wire Line
-	4350 2750 4350 2700
-Wire Wire Line
-	4350 1850 4350 1800
+P 3950 3800
+F 0 "C14" H 4065 3846 50  0000 L CNN
+F 1 "10pC" H 4065 3755 50  0000 L CNN
+F 2 "Capacitor_SMD:C_0805_2012Metric_Pad1.15x1.40mm_HandSolder" H 3988 3650 50  0001 C CNN
+F 3 "~" H 3950 3800 50  0001 C CNN
+F 4 "DNP" H 3950 3800 50  0001 C CNN "Manufacturer Part Number"
+	1    3950 3800
+	1    0    0    -1
+$EndComp
+Text Label 3950 2350 1    50   ~ 0
+GND
+Wire Wire Line
+	3950 2150 3950 2350
+Text Label 3950 3250 1    50   ~ 0
+GND
+Wire Wire Line
+	3950 3050 3950 3250
+Text Label 3950 4150 1    50   ~ 0
+GND
+Wire Wire Line
+	3950 3950 3950 4150
+Wire Wire Line
+	3950 3600 3950 3650
+Wire Wire Line
+	3950 2750 3950 2700
+Wire Wire Line
+	3950 1850 3950 1800
 Wire Wire Line
 	5100 2700 5250 2700
@@
 Wire Wire Line
 	10000 2300 10000 2100
-Wire Wire Line
-	4650 1800 4350 1800
-Connection ~ 4350 1800
-Wire Wire Line
-	4350 2700 4650 2700
-Connection ~ 4350 2700
-Wire Wire Line
-	4650 3600 4350 3600
-Connection ~ 4350 3600
 Text Notes 5850 1000 0    50   ~ 0
 Video filter
@@
 Wire Wire Line
 	2200 6750 2200 6550
+$Comp
+L Device:R R8
+U 1 1 5F688AE7
+P 4350 3800
+F 0 "R8" H 4420 3846 50  0000 L CNN
+F 1 "75R" H 4420 3755 50  0000 L CNN
+F 2 "Resistor_SMD:R_0805_2012Metric_Pad1.15x1.40mm_HandSolder" V 4280 3800 50  0001 C CNN
+F 3 "~" H 4350 3800 50  0001 C CNN
+F 4 "KTR10EZPF75R0" H 4350 3800 50  0001 C CNN "Manufacturer Part Number"
+	1    4350 3800
+	1    0    0    -1
+$EndComp
+Text Label 4350 4150 1    50   ~ 0
+GND
+Wire Wire Line
+	4350 3950 4350 4150
+$Comp
+L Device:R R7
+U 1 1 5F68EF9F
+P 4350 2900
+F 0 "R7" H 4420 2946 50  0000 L CNN
+F 1 "75R" H 4420 2855 50  0000 L CNN
+F 2 "Resistor_SMD:R_0805_2012Metric_Pad1.15x1.40mm_HandSolder" V 4280 2900 50  0001 C CNN
+F 3 "~" H 4350 2900 50  0001 C CNN
+F 4 "KTR10EZPF75R0" H 4350 2900 50  0001 C CNN "Manufacturer Part Number"
+	1    4350 2900
+	1    0    0    -1
+$EndComp
+Text Label 4350 3250 1    50   ~ 0
+GND
+Wire Wire Line
+	4350 3050 4350 3250
+$Comp
+L Device:R R6
+U 1 1 5F695598
+P 4350 2000
+F 0 "R6" H 4420 2046 50  0000 L CNN
+F 1 "75R" H 4420 1955 50  0000 L CNN
+F 2 "Resistor_SMD:R_0805_2012Metric_Pad1.15x1.40mm_HandSolder" V 4280 2000 50  0001 C CNN
+F 3 "~" H 4350 2000 50  0001 C CNN
+F 4 "KTR10EZPF75R0" H 4350 2000 50  0001 C CNN "Manufacturer Part Number"
+	1    4350 2000
+	1    0    0    -1
+$EndComp
+Text Label 4350 2350 1    50   ~ 0
+GND
+Wire Wire Line
+	4350 2150 4350 2350
+Wire Wire Line
+	4350 3600 4350 3650
+Wire Wire Line
+	4350 2700 4350 2750
+Wire Wire Line
+	4350 1800 4350 1850
+Wire Wire Line
+	3350 3600 3950 3600
+Connection ~ 3950 3600
+Wire Wire Line
+	3950 3600 4350 3600
+Connection ~ 4350 3600
+Wire Wire Line
+	4350 3600 4650 3600
+Wire Wire Line
+	3350 2700 3950 2700
+Connection ~ 3950 2700
+Wire Wire Line
+	3950 2700 4350 2700
+Connection ~ 4350 2700
+Wire Wire Line
+	4350 2700 4650 2700
+Wire Wire Line
+	3350 1800 3950 1800
+Connection ~ 3950 1800
+Wire Wire Line
+	3950 1800 4350 1800
+Connection ~ 4350 1800
+Wire Wire Line
+	4350 1800 4650 1800
 $EndSCHEMATC

Commit message: Update Dreamcast_VGA_Adapter.sch
Parts:
- R10, R11, R9: Manufacturer Part Number DNP -> KTR10EZPF5104
Changed lines of the file:
@@
 F 2 "Resistor_SMD:R_0805_2012Metric_Pad1.15x1.40mm_HandSolder" V 5030 2500 50  0001 C CNN
 F 3 "~" H 5100 2500 50  0001 C CNN
-F 4 "DNP" H 5100 2500 50  0001 C CNN "Manufacturer Part Number"
+F 4 "KTR10EZPF5104" H 5100 2500 50  0001 C CNN "Manufacturer Part Number"
 	1    5100 2500
 	1    0    0    -1
@@
 F 2 "Resistor_SMD:R_0805_2012Metric_Pad1.15x1.40mm_HandSolder" V 5030 3400 50  0001 C CNN
 F 3 "~" H 5100 3400 50  0001 C CNN
-F 4 "DNP" H 5100 3400 50  0001 C CNN "Manufacturer Part Number"
+F 4 "KTR10EZPF5104" H 5100 3400 50  0001 C CNN "Manufacturer Part Number"
 	1    5100 3400
 	1    0    0    -1
@@
 F 2 "Resistor_SMD:R_0805_2012Metric_Pad1.15x1.40mm_HandSolder" V 5030 1600 50  0001 C CNN
 F 3 "~" H 5100 1600 50  0001 C CNN
-F 4 "DNP" H 5100 1600 50  0001 C CNN "Manufacturer Part Number"
+F 4 "KTR10EZPF5104" H 5100 1600 50  0001 C CNN "Manufacturer Part Number"
 	1    5100 1600
 	1    0    0    -1

Commit message: Update Dreamcast_VGA_Adapter.sch
Parts:
- C16: Manufacturer Part Number tbd -> CC0805KRX7R9BB103
- FB1: Manufacturer Part Number tbd -> BLM21SP471SH1D
- R4, R5: value 36R -> 39R; Manufacturer Part Number tbd -> RC0805FR-0739RL
Changed lines of the file:
@@
 P 5250 5400
 F 0 "R4" V 5043 5400 50  0000 C CNN
-F 1 "36R" V 5134 5400 50  0000 C CNN
+F 1 "39R" V 5134 5400 50  0000 C CNN
 F 2 "Resistor_SMD:R_0805_2012Metric_Pad1.15x1.40mm_HandSolder" V 5180 5400 50  0001 C CNN
 F 3 "~" H 5250 5400 50  0001 C CNN
-F 4 "tbd" H 5250 5400 50  0001 C CNN "Manufacturer Part Number"
+F 4 "RC0805FR-0739RL" H 5250 5400 50  0001 C CNN "Manufacturer Part Number"
 	1    5250 5400
 	0    1    1    0
@@
 P 5250 6300
 F 0 "R5" V 5043 6300 50  0000 C CNN
-F 1 "36R" V 5134 6300 50  0000 C CNN
+F 1 "39R" V 5134 6300 50  0000 C CNN
 F 2 "Resistor_SMD:R_0805_2012Metric_Pad1.15x1.40mm_HandSolder" V 5180 6300 50  0001 C CNN
 F 3 "~" H 5250 6300 50  0001 C CNN
-F 4 "tbd" H 5250 6300 50  0001 C CNN "Manufacturer Part Number"
+F 4 "RC0805FR-0739RL" H 5250 6300 50  0001 C CNN "Manufacturer Part Number"
 	1    5250 6300
 	0    1    1    0
@@
 F 2 "Inductor_SMD:L_0805_2012Metric_Pad1.15x1.40mm_HandSolder" V 1280 6150 50  0001 C CNN
 F 3 "~" H 1350 6150 50  0001 C CNN
-F 4 "tbd" H 1350 6150 50  0001 C CNN "Manufacturer Part Number"
+F 4 "BLM21SP471SH1D" H 1350 6150 50  0001 C CNN "Manufacturer Part Number"
 	1    1350 6150
 	0    1    1    0
@@
 F 2 "Capacitor_SMD:C_0805_2012Metric_Pad1.15x1.40mm_HandSolder" H 6338 1400 50  0001 C CNN
 F 3 "~" H 6300 1550 50  0001 C CNN
-F 4 "tbd" H 6300 1550 50  0001 C CNN "Manufacturer Part Number"
+F 4 "CC0805KRX7R9BB103" H 6300 1550 50  0001 C CNN "Manufacturer Part Number"
 	1    6300 1550
 	1    0    0    -1

Commit message: Update Dreamcast_VGA_Adapter.sch
Parts:
- added C18, C19, C20: 5pC, Capacitor_SMD:C_0805_2012Metric_Pad1.15x1.40mm_HandSolder, symbol Device:C
- C10, C11, C15, C17, C4, C5, C6, C9: Manufacturer Part Number tbd -> AC0805KRX7R7BB104
- C12, C13, C14: value 10pC -> 5pC; Manufacturer Part Number DNP -> 08055A5R0CAT2A
- C7: Manufacturer Part Number tbd -> CC0805MKX7R7BB105
- R12, R13, R14: Manufacturer Part Number DNP -> RC0805FR-071KL
- R15, R16: Manufacturer Part Number DNP -> RC0805FR-0710KL
Connections:
- wire segments 142 -> 151
Other:
- moved on the sheet: C12, C13, C14

Commit message: Update Dreamcast_VGA_Adapter.sch
Parts:
- removed J3: Conn_01x03, Connector_JST:JST_XH_B3B-XH-A_1x03_P2.50mm_Vertical, symbol Connector_Generic:Conn_01x03
- removed J4, J5: Conn_01x06, Connector_JST:JST_XH_B6B-XH-A_1x06_P2.50mm_Vertical, symbol Connector_Generic:Conn_01x06
- added J3: Conn_01x14, symbol Connector_Generic:Conn_01x14
Connections:
- wire segments 151 -> 150
Changed lines of the file:
@@
 	1    0    0    1
 $EndComp
-Text Label 2300 2850 2    50   ~ 0
+Text Label 1800 2750 2    50   ~ 0
 V-SYNC
-Text Label 2300 3500 2    50   ~ 0
+Text Label 1800 3150 2    50   ~ 0
 DAC_BLUE
-Text Label 2300 3900 2    50   ~ 0
+Text Label 1800 3350 2    50   ~ 0
 DAC_RED
 Wire Wire Line
-	1900 3900 2300 3900
-Wire Wire Line
-	2300 3500 1900 3500
-Wire Wire Line
-	1900 2850 2300 2850
-Wire Wire Line
-	2300 1800 1900 1800
-Text Label 2300 1800 2    50   ~ 0
+	1400 3350 1800 3350
+Wire Wire Line
+	1800 3150 1400 3150
+Wire Wire Line
+	1400 2750 1800 2750
+Wire Wire Line
+	1800 2150 1400 2150
+Text Label 1800 2150 2    50   ~ 0
 AUDIO-R
 Wire Wire Line
-	1900 3700 2300 3700
-Wire Wire Line
-	2300 2950 1900 2950
-Wire Wire Line
-	1900 2000 2300 2000
-Wire Wire Line
-	2300 2450 1900 2450
-Text Label 2300 3700 2    50   ~ 0
+	1400 3250 1800 3250
+Wire Wire Line
+	1800 2850 1400 2850
+Wire Wire Line
+	1400 2250 1800 2250
+Wire Wire Line
+	1800 2950 1400 2950
+Text Label 1800 3250 2    50   ~ 0
 DAC_GREEN
-Text Label 2300 2950 2    50   ~ 0
+Text Label 1800 2850 2    50   ~ 0
 H-SYNC
-Text Label 2300 2000 2    50   ~ 0
+Text Label 1800 2250 2    50   ~ 0
 AUDIO-L
-Text Label 2300 2450 2    50   ~ 0
-GND
-Wire Wire Line
-	2300 3400 1900 3400
-Text Label 2300 3400 2    50   ~ 0
-GND
-Wire Wire Line
-	2300 3600 1900 3600
-Text Label 2300 3600 2    50   ~ 0
-GND
-Wire Wire Line
-	2300 3800 1900 3800
-Text Label 2300 3800 2    50   ~ 0
-GND
-Wire Wire Line
-	2300 1900 1900 1900
-Text Label 2300 1900 2    50   ~ 0
-GND
-$Comp
-L Connector_Generic:Conn_01x06 J5
-U 1 1 5F32E2AB
-P 1700 3700
-F 0 "J5" H 1618 3175 50  0000 C CNN
-F 1 "Conn_01x06" H 1618 3266 50  0000 C CNN
-F 2 "Connector_JST:JST_XH_B6B-XH-A_1x06_P2.50mm_Vertical" H 1700 3700 50  0001 C CNN
-F 3 "http://www.jst-mfg.com/product/pdf/eng/eXH.pdf" H 1700 3700 50  0001 C CNN
-F 4 "B6B-XH-A(LF)(SN)" H 1700 3700 50  0001 C CNN "Manufacturer Part Number"
-	1    1700 3700
-	-1   0    0    1
-$EndComp
-$Comp
-L Connector_Generic:Conn_01x06 J4
-U 1 1 5F335292
-P 1700 2750
-F 0 "J4" H 1618 2225 50  0000 C CNN
-F 1 "Conn_01x06" H 1618 2316 50  0000 C CNN
-F 2 "Connector_JST:JST_XH_B6B-XH-A_1x06_P2.50mm_Vertical" H 1700 2750 50  0001 C CNN
-F 3 "http://www.jst-mfg.com/product/pdf/eng/eXH.pdf" H 1700 2750 50  0001 C CNN
-F 4 "B6B-XH-A(LF)(SN)" H 1700 2750 50  0001 C CNN "Manufacturer Part Number"
-	1    1700 2750
-	-1   0    0    1
-$EndComp
-Text Label 2300 2750 2    50   ~ 0
+Text Label 1800 2950 2    50   ~ 0
+GND
+Wire Wire Line
+	1800 3450 1400 3450
+Wire Wire Line
+	1800 2350 1400 2350
+Text Label 1800 2350 2    50   ~ 0
+GND
+Text Label 1800 2650 2    50   ~ 0
 MODE1
 Wire Wire Line
-	1900 2750 2300 2750
-Wire Wire Line
-	2300 2650 1900 2650
-Text Label 2300 2650 2    50   ~ 0
+	1400 2650 1800 2650
+Wire Wire Line
+	1800 2550 1400 2550
+Text Label 1800 2550 2    50   ~ 0
 MODE2
-Text Label 2300 2550 2    50   ~ 0
+Text Label 1800 2450 2    50   ~ 0
 5V_IN
 Wire Wire Line
-	2300 2550 1900 2550
-$Comp
-L Connector_Generic:Conn_01x03 J3
-U 1 1 5F357949
-P 1700 1900
-F 0 "J3" H 1618 1575 50  0000 C CNN
-F 1 "Conn_01x03" H 1618 1666 50  0000 C CNN
-F 2 "Connector_JST:JST_XH_B3B-XH-A_1x03_P2.50mm_Vertical" H 1700 1900 50  0001 C CNN
-F 3 "http://www.jst-mfg.com/product/pdf/eng/eXH.pdf" H 1700 1900 50  0001 C CNN
-F 4 "B3B-XH-A(LF)(SN)" H 1700 1900 50  0001 C CNN "Manufacturer Part Number"
-	1    1700 1900
-	-1   0    0    1
-$EndComp
+	1800 2450 1400 2450
 $Comp
 L Device:CP C8
@@
 Wire Wire Line
 	3900 3600 3400 3600
+Text Label 1800 3450 2    50   ~ 0
+GND
+$Comp
+L Connector_Generic:Conn_01x14 J3
+U 1 1 5F6E97C2
+P 1200 2850
+F 0 "J3" H 1118 1925 50  0000 C CNN
+F 1 "Conn_01x14" H 1118 2016 50  0000 C CNN
+F 2 "" H 1200 2850 50  0001 C CNN
+F 3 "~" H 1200 2850 50  0001 C CNN
+	1    1200 2850
+	-1   0    0    1
+$EndComp
+Wire Wire Line
+	1800 3050 1400 3050
+Text Label 1800 3050 2    50   ~ 0
+GND
 $EndSCHEMATC

Commit message: Update Dreamcast_VGA_Adapter.sch
Parts:
- removed J3: Conn_01x14, symbol Connector_Generic:Conn_01x14
- added J3: Conn_02x08_Odd_Even, symbol Connector_Generic:Conn_02x08_Odd_Even
Connections:
- wire segments 150 -> 152
Other:
- note added: "Use cable P/N: 3659/16 1000\nhttps://multimedia.3m.com/mws/media/22054O/3mtm-rnd-shld-jckt-flat-cable-mass-term-3659-series-ts0083.pdf"
Changed lines of the file:
@@
 	1    0    0    1
 $EndComp
-Text Label 1800 2750 2    50   ~ 0
+Text Label 900  2950 0    50   ~ 0
 V-SYNC
-Text Label 1800 3150 2    50   ~ 0
+Text Label 2200 3050 2    50   ~ 0
 DAC_BLUE
-Text Label 1800 3350 2    50   ~ 0
+Text Label 2200 3250 2    50   ~ 0
 DAC_RED
 Wire Wire Line
-	1400 3350 1800 3350
-Wire Wire Line
-	1800 3150 1400 3150
-Wire Wire Line
-	1400 2750 1800 2750
-Wire Wire Line
-	1800 2150 1400 2150
-Text Label 1800 2150 2    50   ~ 0
+	1800 3250 2200 3250
+Wire Wire Line
+	2200 3050 1800 3050
+Wire Wire Line
+	1300 2950 900  2950
+Wire Wire Line
+	2200 2550 1800 2550
+Text Label 2200 2550 2    50   ~ 0
 AUDIO-R
 Wire Wire Line
-	1400 3250 1800 3250
-Wire Wire Line
-	1800 2850 1400 2850
-Wire Wire Line
-	1400 2250 1800 2250
-Wire Wire Line
-	1800 2950 1400 2950
-Text Label 1800 3250 2    50   ~ 0
+	1800 3150 2200 3150
+Wire Wire Line
+	2200 2950 1800 2950
+Wire Wire Line
+	1800 2650 2200 2650
+Wire Wire Line
+	900  2650 1300 2650
+Text Label 2200 3150 2    50   ~ 0
 DAC_GREEN
-Text Label 1800 2850 2    50   ~ 0
+Text Label 2200 2950 2    50   ~ 0
 H-SYNC
-Text Label 1800 2250 2    50   ~ 0
+Text Label 2200 2650 2    50   ~ 0
 AUDIO-L
-Text Label 1800 2950 2    50   ~ 0
-GND
-Wire Wire Line
-	1800 3450 1400 3450
-Wire Wire Line
-	1800 2350 1400 2350
-Text Label 1800 2350 2    50   ~ 0
-GND
-Text Label 1800 2650 2    50   ~ 0
+Text Label 900  2650 0    50   ~ 0
+GND
+Wire Wire Line
+	900  2750 1300 2750
+Text Label 900  2750 0    50   ~ 0
+GND
+Text Label 2200 2850 2    50   ~ 0
 MODE1
 Wire Wire Line
-	1400 2650 1800 2650
-Wire Wire Line
-	1800 2550 1400 2550
-Text Label 1800 2550 2    50   ~ 0
+	1800 2850 2200 2850
+Wire Wire Line
+	900  2850 1300 2850
+Text Label 900  2850 0    50   ~ 0
 MODE2
-Text Label 1800 2450 2    50   ~ 0
+Text Label 2200 2750 2    50   ~ 0
 5V_IN
 Wire Wire Line
-	1800 2450 1400 2450
+	2200 2750 1800 2750
 $Comp
 L Device:CP C8
@@
 Wire Wire Line
 	3900 3600 3400 3600
-Text Label 1800 3450 2    50   ~ 0
-GND
-$Comp
-L Connector_Generic:Conn_01x14 J3
-U 1 1 5F6E97C2
-P 1200 2850
-F 0 "J3" H 1118 1925 50  0000 C CNN
-F 1 "Conn_01x14" H 1118 2016 50  0000 C CNN
-F 2 "" H 1200 2850 50  0001 C CNN
-F 3 "~" H 1200 2850 50  0001 C CNN
-	1    1200 2850
-	-1   0    0    1
-$EndComp
-Wire Wire Line
-	1800 3050 1400 3050
-Text Label 1800 3050 2    50   ~ 0
-GND
+Wire Wire Line
+	900  3050 1300 3050
+Text Label 900  3050 0    50   ~ 0
+GND
+Wire Wire Line
+	900  3250 1300 3250
+Text Label 900  3250 0    50   ~ 0
+GND
+Wire Wire Line
+	900  3150 1300 3150
+Text Label 900  3150 0    50   ~ 0
+GND
+Wire Wire Line
+	900  2550 1300 2550
+Text Label 900  2550 0    50   ~ 0
+GND
+$Comp
+L Connector_Generic:Conn_02x08_Odd_Even J3
+U 1 1 5F7CB957
+P 1500 2850
+F 0 "J3" H 1550 3367 50  0000 C CNN
+F 1 "Conn_02x08_Odd_Even" H 1550 3276 50  0000 C CNN
+F 2 "" H 1500 2850 50  0001 C CNN
+F 3 "https://multimedia.3m.com/mws/media/375264O/3mtm-100-in-pcb-100x-100-two-row-78xx-series-ts2104.pdf" H 1500 2850 50  0001 C CNN
+F 4 "7816-0000PR" H 1500 2850 50  0001 C CNN "Manufacturer Part Number"
+	1    1500 2850
+	1    0    0    -1
+$EndComp
+Text Notes 550  700  0    50   ~ 0
+Use cable P/N: 3659/16 1000\nhttps://multimedia.3m.com/mws/media/22054O/3mtm-rnd-shld-jckt-flat-cable-mass-term-3659-series-ts0083.pdf
 $EndSCHEMATC
