File: Hardware/Dreamcast_VGA_Adapter.sch (KiCad schematic (older format))
At the start: 43 parts, among them J1 AudioJack3, J2 DB15_Female_HighDensity_Mount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, J3 Conn_02x08_Odd_Even, SW1 SW_DIP_x02, U1 THS7316, U2 74HCT2G34

Commit message: Update Dreamcast_VGA_Adapter.sch
Parts:
- added C21: 1uC, Capacitor_SMD:C_0805_2012Metric_Pad1.15x1.40mm_HandSolder, symbol Device:C
- C8: value 100uCP -> 33uCP; footprint Capacitor_THT:CP_Radial_D5.0mm_P2.00mm -> Capacitor_Tantalum_SMD:CP_EIA-3528-21_Kemet-B_Pad1.50x2.35mm_HandSolder; Manufacturer Part Number 16ZLH100MEFC5X11 -> TAJB336K006RNJ
Connections:
- net 5V_IN: now also C21.1
- net GND: now also C21.2
Other:
- moved on the sheet: C8
Changed lines of the file:
@@
 L Device:CP C8
 U 1 1 5F681767
-P 2200 6400
-F 0 "C8" H 2318 6446 50  0000 L CNN
-F 1 "100uCP" H 2318 6355 50  0000 L CNN
-F 2 "Capacitor_THT:CP_Radial_D5.0mm_P2.00mm" H 2238 6250 50  0001 C CNN
-F 3 "http://www.rubycon.co.jp/en/catalog/e_pdfs/aluminum/e_zlh.pdf" H 2200 6400 50  0001 C CNN
-F 4 "16ZLH100MEFC5X11" H 2200 6400 50  0001 C CNN "Manufacturer Part Number"
-	1    2200 6400
-	1    0    0    -1
-$EndComp
-Wire Wire Line
-	1650 6150 2200 6150
-Wire Wire Line
-	2200 6250 2200 6150
+P 1150 6400
+F 0 "C8" H 1268 6446 50  0000 L CNN
+F 1 "33uCP" H 1268 6355 50  0000 L CNN
+F 2 "Capacitor_Tantalum_SMD:CP_EIA-3528-21_Kemet-B_Pad1.50x2.35mm_HandSolder" H 1188 6250 50  0001 C CNN
+F 3 "http://datasheets.avx.com/TAJ.pdf" H 1150 6400 50  0001 C CNN
+F 4 "TAJB336K006RNJ" H 1150 6400 50  0001 C CNN "Manufacturer Part Number"
+	1    1150 6400
+	1    0    0    -1
+$EndComp
+Wire Wire Line
+	1150 6250 1150 6150
 Text Label 2900 6150 2    50   ~ 0
 5V
-Text Label 2200 6750 1    50   ~ 0
-GND
-Wire Wire Line
-	2200 6750 2200 6550
+Text Label 1150 6750 1    50   ~ 0
+GND
+Wire Wire Line
+	1150 6750 1150 6550
 $Comp
 L Device:R R8
@@
 Use cable P/N: 3659/16 1000\nhttps://multimedia.3m.com/mws/media/22054O/3mtm-rnd-shld-jckt-flat-cable-mass-term-3659-series-ts0083.pdf
 Wire Wire Line
-	2400 6150 2200 6150
-Connection ~ 2200 6150
-Wire Wire Line
 	2900 6150 2700 6150
+Text Label 700  6150 0    50   ~ 0
+5V_IN
+Wire Wire Line
+	1650 6150 2150 6150
+$Comp
+L Device:C C21
+U 1 1 5F7A229E
+P 2150 6400
+F 0 "C21" H 2265 6446 50  0000 L CNN
+F 1 "1uC" H 2265 6355 50  0000 L CNN
+F 2 "Capacitor_SMD:C_0805_2012Metric_Pad1.15x1.40mm_HandSolder" H 2188 6250 50  0001 C CNN
+F 3 "~" H 2150 6400 50  0001 C CNN
+F 4 "" H 2150 6400 50  0001 C CNN "Manufacturer Part Number"
+	1    2150 6400
+	1    0    0    -1
+$EndComp
+Text Label 2150 6750 1    50   ~ 0
+GND
+Wire Wire Line
+	2150 6750 2150 6550
+Wire Wire Line
+	2150 6250 2150 6150
+Connection ~ 2150 6150
+Wire Wire Line
+	2150 6150 2400 6150
+Wire Wire Line
+	700  6150 1150 6150
 Connection ~ 1650 6150
-Wire Wire Line
-	1350 6150 1650 6150
-Text Label 1350 6150 0    50   ~ 0
-5V_IN
+Connection ~ 1150 6150
+Wire Wire Line
+	1150 6150 1650 6150
 $EndSCHEMATC
