File: Hardware/Dreamcast_VGA_Adapter.sch (KiCad schematic (older format))
At the start: 44 parts, among them J1 AudioJack3, J2 DB15_Female_HighDensity_Mount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, J3 Conn_02x08_Odd_Even, SW1 SW_DIP_x02, U1 THS7316, U2 74HCT2G34

Commit message: Update Dreamcast_VGA_Adapter.sch
Parts:
- C21: Manufacturer Part Number (none) -> CC0805MKX7R7BB105
Changed lines of the file:
@@
 F 2 "Capacitor_SMD:C_0805_2012Metric_Pad1.15x1.40mm_HandSolder" H 2638 6250 50  0001 C CNN
 F 3 "~" H 2600 6400 50  0001 C CNN
-F 4 "" H 2600 6400 50  0001 C CNN "Manufacturer Part Number"
+F 4 "CC0805MKX7R7BB105" H 2600 6400 50  0001 C CNN "Manufacturer Part Number"
 	1    2600 6400
 	1    0    0    -1

Commit message: Progressed circuit design.
Other:
- note added: "Use cable P/N: 3659/16 1000\nhttps://multimedia.3m.com/mws/media/22054O/3mtm-rnd-shld-jckt-flat-cable-mass-term-3659-series-ts0083.pdf\n\nUse box P/N: 1593KBK\nhttp://www.hammondmfg.com/pdf/1593K.pdf"
- note removed: "Use cable P/N: 3659/16 1000\nhttps://multimedia.3m.com/mws/media/22054O/3mtm-rnd-shld-jckt-flat-cable-mass-term-3659-series-ts0083.pdf"
Changed lines of the file:
@@
 	1    0    0    -1
 $EndComp
-Text Notes 550  700  0    50   ~ 0
-Use cable P/N: 3659/16 1000\nhttps://multimedia.3m.com/mws/media/22054O/3mtm-rnd-shld-jckt-flat-cable-mass-term-3659-series-ts0083.pdf
+Text Notes 550  900  0    50   ~ 0
+Use cable P/N: 3659/16 1000\nhttps://multimedia.3m.com/mws/media/22054O/3mtm-rnd-shld-jckt-flat-cable-mass-term-3659-series-ts0083.pdf\n\nUse box P/N: 1593KBK\nhttp://www.hammondmfg.com/pdf/1593K.pdf
 Wire Wire Line
 	1250 6150 1050 6150

Commit message: Progressed circuit design.
Parts:
- J3: footprint (none) -> Connector_IDC:IDC-Header_2x08_P2.54mm_Vertical
Changed lines of the file:
@@
 F 0 "J3" H 1550 3367 50  0000 C CNN
 F 1 "Conn_02x08_Odd_Even" H 1550 3276 50  0000 C CNN
-F 2 "" H 1500 2850 50  0001 C CNN
+F 2 "Connector_IDC:IDC-Header_2x08_P2.54mm_Vertical" H 1500 2850 50  0001 C CNN
 F 3 "https://multimedia.3m.com/mws/media/375264O/3mtm-100-in-pcb-100x-100-two-row-78xx-series-ts2104.pdf" H 1500 2850 50  0001 C CNN
 F 4 "7816-0000PR" H 1500 2850 50  0001 C CNN "Manufacturer Part Number"

Commit message: Progressed circuit design.
Connections:
- net DAC_BLUE: now also C11.2, C14.1, C20.1, J3.16 (Pin_16), R8.1; no longer C10.2, C13.1, C19.1, J3.12 (Pin_12), R7.1
- net DAC_GREEN: now also C10.2, C13.1, C19.1, R7.1; no longer C12.1, C18.1, C9.2, R6.1
- net DAC_RED: now also C12.1, C18.1, C9.2, J3.12 (Pin_12), R6.1; no longer C11.2, C14.1, C20.1, J3.16 (Pin_16), R8.1
- net FILT_BLUE: now also R3.1; no longer R2.1
- net FILT_GREEN: now also R2.1; no longer R1.1
- net FILT_RED: now also R1.1; no longer R3.1
Changed lines of the file:
@@
 Text Label 7050 5400 2    50   ~ 0
 V-SYNC_OUT
+Text Label 8200 3600 2    50   ~ 0
+FILT_BLUE
 Text Label 8200 2700 2    50   ~ 0
-FILT_BLUE
+FILT_GREEN
 Text Label 8200 1800 2    50   ~ 0
-FILT_GREEN
-Text Label 8200 3600 2    50   ~ 0
 FILT_RED
 Text Label 2650 5050 2    50   ~ 0
@@
 	7400 4000 7400 3600
 Wire Wire Line
+	7750 3600 8200 3600
+Wire Wire Line
 	7750 2700 8200 2700
 Wire Wire Line
 	7750 1800 8200 1800
-Wire Wire Line
-	7750 3600 8200 3600
 Wire Wire Line
 	7450 1800 7400 1800
@@
 	1    0    0    -1
 $EndComp
-Text Label 2800 1800 0    50   ~ 0
+Text Label 2800 2700 0    50   ~ 0
 DAC_GREEN
-Text Label 2800 2700 0    50   ~ 0
+Text Label 2800 3600 0    50   ~ 0
 DAC_BLUE
 Text Label 6100 3350 1    50   ~ 0
@@
 Wire Wire Line
 	5100 3100 5100 3250
-Text Label 2800 3600 0    50   ~ 0
+Text Label 2800 1800 0    50   ~ 0
 DAC_RED
 Wire Wire Line
@@
 Text Label 900  2950 0    50   ~ 0
 V-SYNC
+Text Label 2200 3250 2    50   ~ 0
+DAC_BLUE
 Text Label 2200 3050 2    50   ~ 0
-DAC_BLUE
-Text Label 2200 3250 2    50   ~ 0
 DAC_RED
 Wire Wire Line
-	1800 3250 2200 3250
-Wire Wire Line
-	2200 3050 1800 3050
+	1800 3050 2200 3050
+Wire Wire Line
+	2200 3250 1800 3250
 Wire Wire Line
 	1300 2950 900  2950
@@
 	4350 1800 3900 1800
 Connection ~ 4350 1800
-Connection ~ 3400 1800
-Wire Wire Line
-	3400 1800 2800 1800
+Wire Wire Line
+	3400 2700 2800 2700
 Connection ~ 3900 1800
 Wire Wire Line
 	3900 1800 3400 1800
 Wire Wire Line
-	2800 2700 3400 2700
+	2800 3600 3400 3600
 Connection ~ 4350 2700
 Connection ~ 3400 2700
@@
 	4350 3600 3900 3600
 Connection ~ 4350 3600
-Connection ~ 3400 3600
-Wire Wire Line
-	3400 3600 2800 3600
+Wire Wire Line
+	3400 1800 2800 1800
 Connection ~ 3900 3600
 Wire Wire Line
@@
 	1550 6150 1600 6150
 Connection ~ 1600 6150
+Connection ~ 3400 3600
+Connection ~ 3400 1800
 $EndSCHEMATC

Commit message: Progressed circuit design.
Connections:
- net GND: no longer J2.0
- no-connect marks 5 -> 6
Changed lines of the file:
@@
 Wire Wire Line
 	5500 6300 5400 6300
-Text Label 10000 2100 3    50   ~ 0
-GND
-Wire Wire Line
-	10000 2300 10000 2100
 Text Notes 5850 1000 0    50   ~ 0
 Video filter
@@
 Connection ~ 3400 3600
 Connection ~ 3400 1800
+NoConn ~ 10000 2300
 $EndSCHEMATC

Commit message: Progressed circuit design.
Parts:
- removed C12, C13, C14: 5pC, Capacitor_SMD:C_0805_2012Metric_Pad1.15x1.40mm_HandSolder, symbol Device:C
Changed lines of the file:
@@
 	1    0    0    -1
 $EndComp
-Text Label 2800 2700 0    50   ~ 0
+Text Label 3400 2700 0    50   ~ 0
 DAC_GREEN
-Text Label 2800 3600 0    50   ~ 0
+Text Label 3400 3600 0    50   ~ 0
 DAC_BLUE
 Text Label 6100 3350 1    50   ~ 0
@@
 Wire Wire Line
 	5100 3100 5100 3250
-Text Label 2800 1800 0    50   ~ 0
+Text Label 3400 1800 0    50   ~ 0
 DAC_RED
 Wire Wire Line
@@
 	6750 3600 6900 3600
 Connection ~ 6900 3600
-$Comp
-L Device:C C12
-U 1 1 5F1E6679
-P 3400 2000
-F 0 "C12" H 3515 2046 50  0000 L CNN
-F 1 "5pC" H 3515 1955 50  0000 L CNN
-F 2 "Capacitor_SMD:C_0805_2012Metric_Pad1.15x1.40mm_HandSolder" H 3438 1850 50  0001 C CNN
-F 3 "~" H 3400 2000 50  0001 C CNN
-F 4 "08055A5R0CAT2A" H 3400 2000 50  0001 C CNN "Manufacturer Part Number"
-	1    3400 2000
-	1    0    0    -1
-$EndComp
-$Comp
-L Device:C C13
-U 1 1 5F1E76F3
-P 3400 2900
-F 0 "C13" H 3515 2946 50  0000 L CNN
-F 1 "5pC" H 3515 2855 50  0000 L CNN
-F 2 "Capacitor_SMD:C_0805_2012Metric_Pad1.15x1.40mm_HandSolder" H 3438 2750 50  0001 C CNN
-F 3 "~" H 3400 2900 50  0001 C CNN
-F 4 "08055A5R0CAT2A" H 3400 2900 50  0001 C CNN "Manufacturer Part Number"
-	1    3400 2900
-	1    0    0    -1
-$EndComp
-$Comp
-L Device:C C14
-U 1 1 5F1E806E
-P 3400 3800
-F 0 "C14" H 3515 3846 50  0000 L CNN
-F 1 "5pC" H 3515 3755 50  0000 L CNN
-F 2 "Capacitor_SMD:C_0805_2012Metric_Pad1.15x1.40mm_HandSolder" H 3438 3650 50  0001 C CNN
-F 3 "~" H 3400 3800 50  0001 C CNN
-F 4 "08055A5R0CAT2A" H 3400 3800 50  0001 C CNN "Manufacturer Part Number"
-	1    3400 3800
-	1    0    0    -1
-$EndComp
-Text Label 3400 2350 1    50   ~ 0
-GND
-Wire Wire Line
-	3400 2150 3400 2350
-Text Label 3400 3250 1    50   ~ 0
-GND
-Wire Wire Line
-	3400 3050 3400 3250
-Text Label 3400 4150 1    50   ~ 0
-GND
-Wire Wire Line
-	3400 3950 3400 4150
-Wire Wire Line
-	3400 3600 3400 3650
-Wire Wire Line
-	3400 2750 3400 2700
-Wire Wire Line
-	3400 1850 3400 1800
 Wire Wire Line
 	5100 2700 5250 2700
@@
 	4350 1800 3900 1800
 Connection ~ 4350 1800
-Wire Wire Line
-	3400 2700 2800 2700
-Connection ~ 3900 1800
-Wire Wire Line
-	3900 1800 3400 1800
-Wire Wire Line
-	2800 3600 3400 3600
 Connection ~ 4350 2700
-Connection ~ 3400 2700
-Wire Wire Line
-	3400 2700 3900 2700
-Connection ~ 3900 2700
 Wire Wire Line
 	3900 2700 4350 2700
@@
 	4350 3600 3900 3600
 Connection ~ 4350 3600
-Wire Wire Line
-	3400 1800 2800 1800
-Connection ~ 3900 3600
-Wire Wire Line
-	3900 3600 3400 3600
 Wire Wire Line
 	900  3050 1300 3050
@@
 	1550 6150 1600 6150
 Connection ~ 1600 6150
-Connection ~ 3400 3600
-Connection ~ 3400 1800
 NoConn ~ 10000 2300
+Wire Wire Line
+	3900 3600 3400 3600
+Connection ~ 3900 3600
+Wire Wire Line
+	3400 2700 3900 2700
+Connection ~ 3900 2700
+Wire Wire Line
+	3400 1800 3900 1800
+Connection ~ 3900 1800
 $EndSCHEMATC
