File: Hardware/Dreamcast_VGA_Adapter.kicad_pcb (KiCad board)
At the start: 2 copper layers, 56.6 x 57.7 mm, 0 parts

Commit message: Progressed circuit design.
Parts:
- added C1: 470uCP, Capacitor_THT:CP_Radial_D8.0mm_P3.50mm, F.Cu at (53.0, 7.00)
- added C10: 0.1uC, Capacitor_SMD:C_0805_2012Metric_Pad1.15x1.40mm_HandSolder, F.Cu at (70.3, 11.0)
- added C11: 0.1uC, Capacitor_SMD:C_0805_2012Metric_Pad1.15x1.40mm_HandSolder, F.Cu at (111.9, -23.4)
- added C12: 5pC, Capacitor_SMD:C_0805_2012Metric_Pad1.15x1.40mm_HandSolder, F.Cu at (110.1, -4.79)
- added C13: 5pC, Capacitor_SMD:C_0805_2012Metric_Pad1.15x1.40mm_HandSolder, F.Cu at (75.1, 11.0)
- added C14: 5pC, Capacitor_SMD:C_0805_2012Metric_Pad1.15x1.40mm_HandSolder, F.Cu at (79.8, 6.65)
- added C15: 0.1uC, Capacitor_SMD:C_0805_2012Metric_Pad1.15x1.40mm_HandSolder, F.Cu at (106.1, -19.5)
- added C16: 0.01uC, Capacitor_SMD:C_0805_2012Metric_Pad1.15x1.40mm_HandSolder, F.Cu at (95.8, -0.39)
- added C17: 0.1uC, Capacitor_SMD:C_0805_2012Metric_Pad1.15x1.40mm_HandSolder, F.Cu at (110.8, -19.5)
- added C18: 5pC, Capacitor_SMD:C_0805_2012Metric_Pad1.15x1.40mm_HandSolder, F.Cu at (106.1, -16.6)
- added C19: 5pC, Capacitor_SMD:C_0805_2012Metric_Pad1.15x1.40mm_HandSolder, F.Cu at (84.6, 6.46)
- added C2: 470uCP, Capacitor_THT:CP_Radial_D8.0mm_P3.50mm, F.Cu at (74.2, -2.55)
- added C20: 5pC, Capacitor_SMD:C_0805_2012Metric_Pad1.15x1.40mm_HandSolder, F.Cu at (79.8, 9.60)
- added C21: 1uC, Capacitor_SMD:C_0805_2012Metric_Pad1.15x1.40mm_HandSolder, F.Cu at (106.1, -13.6)
- added C3: 470uCP, Capacitor_THT:CP_Radial_D8.0mm_P3.50mm, F.Cu at (64.4, -2.55)
- added C4: 0.1uC, Capacitor_SMD:C_0805_2012Metric_Pad1.15x1.40mm_HandSolder, F.Cu at (100.6, 5.51)
- added C5: 0.1uC, Capacitor_SMD:C_0805_2012Metric_Pad1.15x1.40mm_HandSolder, F.Cu at (89.3, 9.41)
- added C6: 0.1uC, Capacitor_SMD:C_0805_2012Metric_Pad1.15x1.40mm_HandSolder, F.Cu at (76.7, 3.70)
- added C7: 1uC, Capacitor_SMD:C_0805_2012Metric_Pad1.15x1.40mm_HandSolder, F.Cu at (95.8, -3.34)
- added C8: 33uCP, Capacitor_Tantalum_SMD:CP_EIA-3528-21_Kemet-B_Pad1.50x2.35mm_HandSolder, F.Cu at (71.2, 4.40)
- added C9: 0.1uC, Capacitor_SMD:C_0805_2012Metric_Pad1.15x1.40mm_HandSolder, F.Cu at (75.1, 8.05)
- added FB1: Ferrite_Bead, Inductor_SMD:L_0805_2012Metric_Pad1.15x1.40mm_HandSolder, F.Cu at (70.3, 8.05)
- added J1: AudioJack3, Connector_Audio_custom:Jack_3.5mm_CUI_SJ1-3533NG_Horizontal, F.Cu at (-21.5, 26.3)
- added J2: DB15_Female_HighDensity_MountingHoles, Connector_Dsub_custom:DSUB-15-HD_Female_Horizontal_P2.29x1.98mm_EdgePinOffset3.03mm_Housed_MountingHolesOffset4.94mm, F.Cu at (4.33, 21.8)
- added J3: Conn_02x08_Odd_Even, Connector_IDC:IDC-Header_2x08_P2.54mm_Vertical, F.Cu at (8.89, -23.8)
- added R1: 75R, Resistor_SMD:R_0805_2012Metric_Pad1.15x1.40mm_HandSolder, F.Cu at (106.1, -10.7)
- added R10: 5.1MR, Resistor_SMD:R_0805_2012Metric_Pad1.15x1.40mm_HandSolder, F.Cu at (110.8, -16.6)
- added R11: 5.1MR, Resistor_SMD:R_0805_2012Metric_Pad1.15x1.40mm_HandSolder, F.Cu at (105.3, -3.34)
- added R12: 1kR, Resistor_SMD:R_0805_2012Metric_Pad1.15x1.40mm_HandSolder, F.Cu at (95.8, 5.51)
- added R13: 1kR, Resistor_SMD:R_0805_2012Metric_Pad1.15x1.40mm_HandSolder, F.Cu at (100.6, 2.56)
- added R14: 1kR, Resistor_SMD:R_0805_2012Metric_Pad1.15x1.40mm_HandSolder, F.Cu at (110.8, -7.74)
- added R15: 10kR, Resistor_SMD:R_0805_2012Metric_Pad1.15x1.40mm_HandSolder, F.Cu at (105.3, -0.39)
- added R16: 10kR, Resistor_SMD:R_0805_2012Metric_Pad1.15x1.40mm_HandSolder, F.Cu at (94.1, 8.46)
- added R2: 75R, Resistor_SMD:R_0805_2012Metric_Pad1.15x1.40mm_HandSolder, F.Cu at (84.6, 9.41)
- added R3: 75R, Resistor_SMD:R_0805_2012Metric_Pad1.15x1.40mm_HandSolder, F.Cu at (89.3, 6.46)
- added R4: 39R, Resistor_SMD:R_0805_2012Metric_Pad1.15x1.40mm_HandSolder, F.Cu at (95.8, 2.56)
- added R5: 39R, Resistor_SMD:R_0805_2012Metric_Pad1.15x1.40mm_HandSolder, F.Cu at (106.1, -7.74)
- added R6: 75R, Resistor_SMD:R_0805_2012Metric_Pad1.15x1.40mm_HandSolder, F.Cu at (110.8, -13.6)
- added R7: 75R, Resistor_SMD:R_0805_2012Metric_Pad1.15x1.40mm_HandSolder, F.Cu at (100.6, -0.39)
- added R8: 75R, Resistor_SMD:R_0805_2012Metric_Pad1.15x1.40mm_HandSolder, F.Cu at (110.8, -10.7)
- added R9: 5.1MR, Resistor_SMD:R_0805_2012Metric_Pad1.15x1.40mm_HandSolder, F.Cu at (100.6, -3.34)
- added SW1: SW_DIP_x02, Button_Switch_THT:SW_DIP_SPSTx02_Slide_9.78x7.26mm_W7.62mm_P2.54mm, F.Cu at (51.7, -4.10)
- added U1: THS7316, Package_SO:SOIC-8_3.9x4.9mm_P1.27mm, F.Cu at (63.7, 8.21)
- added U2: 74HCT2G34, Package_TO_SOT_SMD:SOT-363_SC-70-6_Handsoldering, F.Cu at (106.6, -22.9)

Commit message: Progressed circuit design.
Parts:
- moved J1 44.5 mm to (23.0, 26.3)

Commit message: Progressed circuit design.
Parts:
- C4, C5, C6: moved to B.Cu
- moved R14 130.9 mm to (-20.0, -4.00), turned to 90 degrees
- moved C11 118.5 mm to (-6.00, -12.0), turned to 90 degrees
- moved R1 103.3 mm to (6.00, 15.0), turned to 90 degrees
- moved R3 95.7 mm to (-6.00, 15.0), turned to 90 degrees
- moved C4 93.6 mm to (7.00, 6.97), turned to 90 degrees
- moved C5 91.4 mm to (-2.00, 7.00), turned to 90 degrees
- moved C6 87.7 mm to (-11.0, 7.00), turned to 90 degrees
- moved R2 84.8 mm to (0.00, 15.0), turned to 90 degrees
- moved SW1 75.5 mm to (-21.2, -23.8), turned to 270 degrees
- moved C10 75.0 mm to (-1.00, -12.0), turned to 90 degrees
- moved C2 74.6 mm to (-0.10, 5.00), turned to 270 degrees
- moved C3 73.8 mm to (-9.00, 5.00), turned to 270 degrees
- moved C9 72.9 mm to (5.00, -12.0), turned to 90 degrees
- moved U1 64.3 mm to (0.80, -4.90), turned to 270 degrees
- moved C1 44.0 mm to (9.00, 5.00), turned to 270 degrees
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Connections:
- C10 pad 2: /DAC_BLUE -> /DAC_GREEN
- C11 pad 2: /DAC_RED -> /DAC_BLUE
- C12 pad 1: /DAC_GREEN -> /DAC_RED
- C13 pad 1: /DAC_BLUE -> /DAC_GREEN
- C14 pad 1: /DAC_RED -> /DAC_BLUE
- C18 pad 1: /DAC_GREEN -> /DAC_RED
- C19 pad 1: /DAC_BLUE -> /DAC_GREEN
- C20 pad 1: /DAC_RED -> /DAC_BLUE
- C9 pad 2: /DAC_GREEN -> /DAC_RED
- J3 pad 12: /DAC_BLUE -> /DAC_RED
- J3 pad 16: /DAC_RED -> /DAC_BLUE
- R1 pad 1: /FILT_GREEN -> /FILT_RED
- R2 pad 1: /FILT_BLUE -> /FILT_GREEN
- R3 pad 1: /FILT_RED -> /FILT_BLUE
- R6 pad 1: /DAC_GREEN -> /DAC_RED
- R7 pad 1: /DAC_BLUE -> /DAC_GREEN
- R8 pad 1: /DAC_RED -> /DAC_BLUE
Other:
- net class 75ohm_track added: clearance 0.25, trace_width 1, via_dia 0.8, via_drill 0.4
- net class Default: clearance 0.2 -> 0.25; trace_width 0.25 -> 0.5
- net class Power added: clearance 0.25, trace_width 1, via_dia 0.8, via_drill 0.4
- rule pad_to_mask_clearance: 0.051 -> 0
- rule trace_clearance: 0.2 -> 0.25
- rule trace_min: 0.2 -> 0.1524
- rule via_min_drill: 0.3 -> 0.33
- rule via_min_size: 0.4 -> 0.508

Commit message: Progressed circuit design.
Parts:
- moved U1 0.80 mm to (0.00, -4.90)
Connections:
- J2 pad 0: GND -> Net-(J2-Pad0)
Routing:
- net /AUDIO-L: track 0.00 -> 51.5 mm
- net /AUDIO-R: track 0.00 -> 45.0 mm
- net Net-(C3-Pad1): track 0.00 -> 14.4 mm
- net Net-(C1-Pad1): track 0.00 -> 13.3 mm
- net Net-(C2-Pad1): track 0.00 -> 10.0 mm
- net Net-(C1-Pad2): track 0.00 -> 8.92 mm
- net Net-(C3-Pad2): track 0.00 -> 8.91 mm
- net Net-(C2-Pad2): track 0.00 -> 7.61 mm
- net /FILT_RED: track 0.00 -> 7.43 mm
- net /FILT_BLUE: track 0.00 -> 7.19 mm
- net /FILT_GREEN: track 0.00 -> 5.90 mm
- net GND: vias 0 -> 52
- added copper zone on B.Cu, net GND
- added copper zone on F.Cu, net GND
Changed lines of the file:
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@@
     (thickness 1.6)
     (drawings 16)
-    (tracks 0)
+    (tracks 97)
     (zones 0)
     (modules 44)
-    (nets 34)
+    (nets 35)
   )
   (page A4)
@@
   (net 32 "Net-(R4-Pad1)")
   (net 33 "Net-(R5-Pad1)")
+  (net 34 "Net-(J2-Pad0)")
   (net_class Default "This is the default net class."
     (clearance 0.25)
@@
     (add_net /V-SYNC)
     (add_net /V-SYNC_OUT)
-    (add_net "Net-(C2-Pad2)")
-    (add_net "Net-(C3-Pad2)")
+    (add_net "Net-(J2-Pad0)")
     (add_net "Net-(J2-Pad11)")
     (add_net "Net-(J2-Pad12)")
@@
     (add_net "Net-(C11-Pad1)")
     (add_net "Net-(C2-Pad1)")
+    (add_net "Net-(C2-Pad2)")
     (add_net "Net-(C3-Pad1)")
+    (add_net "Net-(C3-Pad2)")
     (add_net "Net-(C9-Pad1)")
   )
@@
   )
   (module Package_SO:SOIC-8_3.9x4.9mm_P1.27mm (layer F.Cu)
-    (at 0.8 -4.9 270)
+    (at 0 -4.9 270)
     (descr "SOIC, 8 Pin (JEDEC MS-012AA, https://www.analog.com/media/en/package-pcb-resources/package/pkg_pdf/soic_narrow-r/r_8.pdf), generated with kicad-footprint-generator ipc_gullwing_generator.py")
     (tags "SOIC SO")
@@
     (fp_arc (start -16.815 2.05) (end -18.415 2.05) (angle 180) (layer F.Fab) (width 0.1))
     (pad 0 thru_hole circle (at 8.185 2.05) (size 4 4) (drill 3.05) (layers *.Cu *.Mask)
-      (net 7 GND))
+      (net 34 "Net-(J2-Pad0)"))
     (pad 0 thru_hole circle (at -16.815 2.05) (size 4 4) (drill 3.05) (layers *.Cu *.Mask)
-      (net 7 GND))
+      (net 34 "Net-(J2-Pad0)"))
     (pad 15 thru_hole circle (at -9.16 3.96) (size 1.6 1.6) (drill 1.09) (layers *.Cu *.Mask)
       (net 18 "Net-(J2-Pad15)"))
@@
   (gr_line (start 28.305 -28.83) (end -28.305 -28.83) (layer Edge.Cuts) (width 0.05))
   (gr_line (start -28.305 28.83) (end 28.305 28.83) (layer Edge.Cuts) (width 0.05))
+  (via (at -20 -5) (size 0.8) (drill 0.4) (layers F.Cu B.Cu) (net 7))
+  (segment (start 6 11.5) (end 9 8.5) (width 1) (layer F.Cu) (net 1))
+  (segment (start 6 13.975) (end 6 11.5) (width 1) (layer F.Cu) (net 1))
+  (segment (start 8.5 8) (end 9 8.5) (width 1) (layer B.Cu) (net 1))
+  (segment (start 7 8) (end 8.5 8) (width 1) (layer B.Cu) (net 1))
+  (segment (start 8.05 5.95) (end 9 5) (width 1) (layer B.Cu) (net 2))
+  (segment (start 7 5.95) (end 8.05 5.95) (width 1) (layer B.Cu) (net 2))
+  (segment (start 1.905 -1.095) (end 1.905 -2.425) (width 1) (layer F.Cu) (net 2))
+  (segment (start 8 5) (end 1.905 -1.095) (width 1) (layer F.Cu) (net 2))
+  (segment (start 9 5) (end 8 5) (width 1) (layer F.Cu) (net 2))
+  (segment (start 0 8.6) (end -0.1 8.5) (width 1) (layer F.Cu) (net 3))
+  (segment (start 0 13.975) (end 0 8.6) (width 1) (layer F.Cu) (net 3))
+  (segment (start -0.575 8.025) (end -0.1 8.5) (width 1) (layer B.Cu) (net 3))
+  (segment (start -2 8.025) (end -0.575 8.025) (width 1) (layer B.Cu) (net 3))
+  (segment (start -1.075 5.975) (end -0.1 5) (width 1) (layer B.Cu) (net 4))
+  (segment (start -2 5.975) (end -1.075 5.975) (width 1) (layer B.Cu) (net 4))
+  (segment (start 0.635 4.265) (end -0.1 5) (width 1) (layer F.Cu) (net 4))
+  (segment (start 0.635 -2.425) (end 0.635 4.265) (width 1) (layer F.Cu) (net 4))
+  (segment (start -6 11.5) (end -9 8.5) (width 1) (layer F.Cu) (net 5))
+  (segment (start -6 13.975) (end -6 11.5) (width 1) (layer F.Cu) (net 5))
+  (segment (start -9.475 8.025) (end -9 8.5) (width 1) (layer B.Cu) (net 5))
+  (segment (start -11 8.025) (end -9.475 8.025) (width 1) (layer B.Cu) (net 5))
+  (segment (start -9.975 5.975) (end -9 5) (width 1) (layer B.Cu) (net 6))
+  (segment (start -11 5.975) (end -9.975 5.975) (width 1) (layer B.Cu) (net 6))
+  (segment (start -7.082192 5) (end -9 5) (width 1) (layer F.Cu) (net 6))
+  (segment (start -0.635 -1.447192) (end -7.082192 5) (width 1) (layer F.Cu) (net 6))
+  (segment (start -0.635 -2.425) (end -0.635 -1.447192) (width 1) (layer F.Cu) (net 6))
+  (via (at -3 12) (size 0.8) (drill 0.4) (layers F.Cu B.Cu) (net 7))
+  (via (at -3 13.5) (size 0.8) (drill 0.4) (layers F.Cu B.Cu) (net 7))
+  (via (at -3 15) (size 0.8) (drill 0.4) (layers F.Cu B.Cu) (net 7))
+  (via (at -3 16.5) (size 0.8) (drill 0.4) (layers F.Cu B.Cu) (net 7))
+  (via (at 3 12) (size 0.8) (drill 0.4) (layers F.Cu B.Cu) (net 7))
+  (via (at 3 13.5) (size 0.8) (drill 0.4) (layers F.Cu B.Cu) (net 7))
+  (via (at 3 15) (size 0.8) (drill 0.4) (layers F.Cu B.Cu) (net 7))
+  (via (at 3 16.5) (size 0.8) (drill 0.4) (layers F.Cu B.Cu) (net 7))
+  (via (at 9.5 12) (size 0.8) (drill 0.4) (layers F.Cu B.Cu) (net 7))
+  (via (at 9.5 13.5) (size 0.8) (drill 0.4) (layers F.Cu B.Cu) (net 7))
+  (via (at 9.5 15) (size 0.8) (drill 0.4) (layers F.Cu B.Cu) (net 7))
+  (via (at 9.5 16.5) (size 0.8) (drill 0.4) (layers F.Cu B.Cu) (net 7))
+  (via (at -9 12) (size 0.8) (drill 0.4) (layers F.Cu B.Cu) (net 7))
+  (via (at -9 13.5) (size 0.8) (drill 0.4) (layers F.Cu B.Cu) (net 7))
+  (via (at -9 15) (size 0.8) (drill 0.4) (layers F.Cu B.Cu) (net 7))
+  (via (at -9 16.5) (size 0.8) (drill 0.4) (layers F.Cu B.Cu) (net 7))
+  (via (at -3 4) (size 0.8) (drill 0.4) (layers F.Cu B.Cu) (net 7))
+  (via (at 3 4) (size 0.8) (drill 0.4) (layers F.Cu B.Cu) (net 7))
+  (via (at -25 25) (size 0.8) (drill 0.4) (layers F.Cu B.Cu) (net 7))
+  (via (at -25 20) (size 0.8) (drill 0.4) (layers F.Cu B.Cu) (net 7))
+  (via (at -25 15) (size 0.8) (drill 0.4) (layers F.Cu B.Cu) (net 7))
+  (via (at -25 10) (size 0.8) (drill 0.4) (layers F.Cu B.Cu) (net 7))
+  (via (at -25 5) (size 0.8) (drill 0.4) (layers F.Cu B.Cu) (net 7))
+  (via (at -25 0) (size 0.8) (drill 0.4) (layers F.Cu B.Cu) (net 7))
+  (via (at -20 25) (size 0.8) (drill 0.4) (layers F.Cu B.Cu) (net 7))
+  (via (at -10 25) (size 0.8) (drill 0.4) (layers F.Cu B.Cu) (net 7))
+  (via (at 5 25) (size 0.8) (drill 0.4) (layers F.Cu B.Cu) (net 7))
+  (via (at 15 25) (size 0.8) (drill 0.4) (layers F.Cu B.Cu) (net 7))
+  (via (at 25 20) (size 0.8) (drill 0.4) (layers F.Cu B.Cu) (net 7))
+  (via (at 25 15) (size 0.8) (drill 0.4) (layers F.Cu B.Cu) (net 7))
+  (via (at 25 5) (size 0.8) (drill 0.4) (layers F.Cu B.Cu) (net 7))
+  (via (at 25 10) (size 0.8) (drill 0.4) (layers F.Cu B.Cu) (net 7))
+  (via (at 25 0) (size 0.8) (drill 0.4) (layers F.Cu B.Cu) (net 7))
+  (via (at -20 -0.5) (size 0.8) (drill 0.4) (layers F.Cu B.Cu) (net 7))
+  (via (at -20 -10) (size 0.8) (drill 0.4) (layers F.Cu B.Cu) (net 7))
+  (via (at 20 -0.5) (size 0.8) (drill 0.4) (layers F.Cu B.Cu) (net 7))
+  (via (at 20 -5) (size 0.8) (drill 0.4) (layers F.Cu B.Cu) (net 7))
+  (via (at 20 -10) (size 0.8) (drill 0.4) (layers F.Cu B.Cu) (net 7))
+  (via (at 20 -15) (size 0.8) (drill 0.4) (layers F.Cu B.Cu) (net 7))
+  (via (at 25 -15) (size 0.8) (drill 0.4) (layers F.Cu B.Cu) (net 7))
+  (via (at 25 -20) (size 0.8) (drill 0.4) (layers F.Cu B.Cu) (net 7))
+  (via (at 25 -25) (size 0.8) (drill 0.4) (layers F.Cu B.Cu) (net 7))
+  (via (at 20.5 10) (size 0.8) (drill 0.4) (layers F.Cu B.Cu) (net 7))
+  (via (at 20.5 15) (size 0.8) (drill 0.4) (layers F.Cu B.Cu) (net 7))
+  (via (at 20.5 5) (size 0.8) (drill 0.4) (layers F.Cu B.Cu) (net 7))
+  (via (at 17.5 2) (size 0.8) (drill 0.4) (layers F.Cu B.Cu) (net 7))
+  (via (at 14.5 -1) (size 0.8) (drill 0.4) (layers F.Cu B.Cu) (net 7))
+  (via (at 11.5 -4) (size 0.8) (drill 0.4) (layers F.Cu B.Cu) (net 7))
+  (via (at 9.5 -7.5) (size 0.8) (drill 0.4) (layers F.Cu B.Cu) (net 7))
+  (via (at 9.5 -12.5) (size 0.8) (drill 0.4) (layers F.Cu B.Cu) (net 7))
+  (via (at 9.5 -17) (size 0.8) (drill 0.4) (layers F.Cu B.Cu) (net 7))
+  (segment (start 21.7 18.4) (end 21.7 4.2) (width 1) (layer F.Cu) (net 16))
+  (segment (start 21.7 4.2) (end 11 -6.5) (width 1) (layer F.Cu) (net 16))
+  (segment (start 11 -19.15) (end 8.89 -21.26) (width 1) (layer F.Cu) (net 16))
+  (segment (start 11 -6.5) (end 11 -19.15) (width 1) (layer F.Cu) (net 16))
+  (segment (start 21.7 23.9) (end 19 21.2) (width 1) (layer F.Cu) (net 17))
+  (segment (start 19 21.2) (end 19 6) (width 1) (layer F.Cu) (net 17))
+  (segment (start 19 6) (end 8 -5) (width 1) (layer F.Cu) (net 17))
+  (segment (start 8 -5) (end 8 -17) (width 1) (layer F.Cu) (net 17))
+  (segment (start 6.35 -18.65) (end 6.35 -21.26) (width 1) (layer F.Cu) (net 17))
+  (segment (start 8 -17) (end 6.35 -18.65) (width 1) (layer F.Cu) (net 17))
+  (segment (start -6 17) (end -6 16.025) (width 1) (layer F.Cu) (net 25))
+  (segment (start -2.58 20.42) (end -6 17) (width 1) (layer F.Cu) (net 25))
+  (segment (start -2.58 21.8) (end -2.58 20.42) (width 1) (layer F.Cu) (net 25))
+  (segment (start 0 20.42) (end 0 16.025) (width 1) (layer F.Cu) (net 26))
+  (segment (start -0.29 20.71) (end 0 20.42) (width 1) (layer F.Cu) (net 26))
+  (segment (start -0.29 21.8) (end -0.29 20.71) (width 1) (layer F.Cu) (net 26))
+  (segment (start 2 21.0125) (end 6 17.0125) (width 1) (layer F.Cu) (net 27))
+  (segment (start 6 17.0125) (end 6 16.025) (width 1) (layer F.Cu) (net 27))
+  (segment (start 2 21.8) (end 2 21.0125) (width 1) (layer F.Cu) (net 27))
+  (zone (net 7) (net_name GND) (layer F.Cu) (hatch edge 0.508)
+    (connect_pads (clearance 0.508))
+    (min_thickness 0.254)
+    (fill yes (arc_segments 32) (thermal_gap 0.508) (thermal_bridge_width 0.508) (smoothing fillet) (radius 1))
+    (polygon
+      (pts
+        (xy 28.3 28.82) (xy -28.3 28.82) (xy -28.3 -28.83) (xy 28.3 -28.83)
+      )
+    )
+  )
+  (zone (net 7) (net_name GND) (layer B.Cu) (hatch edge 0.508)
+    (connect_pads (clearance 0.508))
+    (min_thickness 0.254)
+    (fill yes (arc_segments 32) (thermal_gap 0.508) (thermal_bridge_width 0.508) (smoothing fillet) (radius 1))
+    (polygon
+      (pts
+        (xy 28.3 28.82) (xy -28.3 28.82) (xy -28.3 -28.83) (xy 28.3 -28.83)
+      )
+    )
+  )
 )

Commit message: Progressed circuit design.
Parts:
- moved R1 3.61 mm to (3.00, 17.0)
- moved R3 3.61 mm to (-3.00, 17.0)
- moved R14 2.90 mm to (-17.1, -4.10)
- moved R2 2.00 mm to (0.00, 17.0)
Routing:
- net /AUDIO-L: track 51.5 -> 0.00 mm
- net /AUDIO-R: track 45.0 -> 0.00 mm
- net Net-(C3-Pad1): track 14.4 -> 0.00 mm
- net Net-(C1-Pad1): track 13.3 -> 0.00 mm
- net Net-(C2-Pad1): track 10.0 -> 0.00 mm
- net Net-(C1-Pad2): track 8.92 -> 0.00 mm
- net Net-(C3-Pad2): track 8.91 -> 0.00 mm
- net Net-(C2-Pad2): track 7.61 -> 0.00 mm
- net /FILT_RED: track 7.43 -> 0.00 mm
- net /FILT_BLUE: track 7.19 -> 0.00 mm
- net /FILT_GREEN: track 5.90 -> 0.00 mm
- net GND: vias 52 -> 27

Commit message: Update Dreamcast_VGA_Adapter.kicad_pcb
Parts:
- removed C12, C13, C14: 5pC, Capacitor_SMD:C_0805_2012Metric_Pad1.15x1.40mm_HandSolder
- R12, R13, R14: moved to B.Cu
- moved C17 152.8 mm to (-41.7, -10.4)
- moved C21 152.8 mm to (-46.5, -4.49)
- moved U2 134.3 mm to (-23.0, 12.0), turned to 270 degrees
- moved R5 130.3 mm to (-23.5, 6.00), turned to 90 degrees
- moved C15 130.0 mm to (-20.0, 12.0), turned to 90 degrees
- moved R15 126.6 mm to (-20.0, 17.5), turned to 180 degrees
- moved R16 118.4 mm to (-24.0, 17.5)
- moved R4 116.9 mm to (-21.0, 6.00), turned to 90 degrees
- moved R8 116.4 mm to (-5.50, -15.0), turned to 180 degrees
- moved C8 114.1 mm to (-42.9, 5.95)
- moved FB1 114.1 mm to (-43.8, 9.60)
- moved R10 112.1 mm to (-1.00, -8.50), turned to 270 degrees
- moved R11 111.9 mm to (-6.50, -8.50), turned to 270 degrees
- moved R6 105.3 mm to (5.50, -15.0), turned to 180 degrees
- moved C7 102.3 mm to (-6.50, -1.50), turned to 270 degrees
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Routing:
- net /H-SYNC: track 0.00 -> 53.0 mm
- net /AUDIO-L: track 0.00 -> 51.7 mm
- net /AUDIO-R: track 0.00 -> 47.2 mm
- net /V-SYNC: track 0.00 -> 45.8 mm
- net /MODE1: track 0.00 -> 32.4 mm
- net /H-SYNC_OUT: track 0.00 -> 30.6 mm
- net /MODE2: track 0.00 -> 24.8 mm
- net GND: track 0.00 -> 23.9 mm, vias 27 -> 69
- net /V-SYNC_OUT: track 0.00 -> 23.8 mm
- net VCC: track 0.00 -> 22.3 mm
- net /DAC_RED: track 0.00 -> 19.3 mm
- net /DAC_GREEN: track 0.00 -> 16.5 mm
- net Net-(C1-Pad2): track 0.00 -> 14.8 mm
- net /DAC_BLUE: track 0.00 -> 14.1 mm
- net Net-(C3-Pad1): track 0.00 -> 13.1 mm
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
Commit message: Update Dreamcast_VGA_Adapter.kicad_pcb
Parts:
- moved FB1 58.6 mm to (12.0, -8.50), turned to 90 degrees
- moved C21 58.6 mm to (12.0, -1.50), turned to 270 degrees
- moved C17 55.0 mm to (13.0, -5.00)
- moved C8 52.4 mm to (9.00, -1.00), turned to 270 degrees
- moved C7 2.80 mm to (-6.00, -4.25), turned to 180 degrees
- moved C16 1.82 mm to (-6.00, -2.00), turned to 180 degrees
Routing:
- net VCC: track 22.3 -> 97.5 mm
- net /5V_IN: track 0.00 -> 15.1 mm
- net /AUDIO-L: track 51.7 -> 56.2 mm
- net /AUDIO-R: track 47.2 -> 51.4 mm
- net GND: track 23.9 -> 26.9 mm, vias 69 -> 75
