File: Hardware/Dreamcast_VGA_Adapter.kicad_pcb (KiCad board)
At the start: 2 copper layers, 56.6 x 57.7 mm, 41 parts, among them J1 AudioJack3, J2 DB15_Female_HighDensity_Mount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, J3 Conn_02x08_Odd_Even, SW1 SW_DIP_x02, U1 THS7316, U2 74HCT2G34

Commit message: Update Dreamcast_VGA_Adapter.kicad_pcb
Parts:
- moved C19 2.25 mm to (0.00, -12.8)
- moved R7 2.25 mm to (0.00, -15.0)
Routing:
- net GND: vias 75 -> 76
Other:
- board text added: "Nuno Sousa 10/2020"
Changed lines of the file:
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@@
   (general
     (thickness 1.6)
-    (drawings 20)
-    (tracks 320)
+    (drawings 30)
+    (tracks 321)
     (zones 0)
     (modules 41)
@@
     (last_trace_width 0.5)
     (trace_clearance 0.25)
-    (zone_clearance 0.508)
+    (zone_clearance 0.254)
     (zone_45_only no)
     (trace_min 0.1524)
@@
     (tags "SOT-363 SC-70-6 Handsoldering")
     (attr smd)
-    (fp_text reference U2 (at 0 -2 90) (layer F.SilkS)
+    (fp_text reference U2 (at 0 2.1 90) (layer F.SilkS)
       (effects (font (size 1 1) (thickness 0.15)))
     )
@@
     (tags "resistor handsolder")
     (attr smd)
-    (fp_text reference R11 (at 0 -1.65 90) (layer F.SilkS)
+    (fp_text reference R11 (at 0 2.9 90) (layer F.SilkS)
       (effects (font (size 1 1) (thickness 0.15)))
     )
@@
     (tags "resistor handsolder")
     (attr smd)
-    (fp_text reference R10 (at 0 -1.65 90) (layer F.SilkS)
+    (fp_text reference R10 (at 3.5 -4.4 90) (layer F.SilkS)
       (effects (font (size 1 1) (thickness 0.15)))
     )
@@
     (tags "resistor handsolder")
     (attr smd)
-    (fp_text reference R9 (at 0 -1.65 90) (layer F.SilkS)
+    (fp_text reference R9 (at 0 -4.2 90) (layer F.SilkS)
       (effects (font (size 1 1) (thickness 0.15)))
     )
@@
     (tags "resistor handsolder")
     (attr smd)
-    (fp_text reference R8 (at 0 -1.65) (layer F.SilkS)
+    (fp_text reference R8 (at 0 1.5) (layer F.SilkS)
       (effects (font (size 1 1) (thickness 0.15)))
     )
@@
   )
   (module Resistor_SMD:R_0805_2012Metric_Pad1.15x1.40mm_HandSolder (layer F.Cu)
-    (at 0 -12.75 180)
+    (at 0 -15 180)
     (descr "Resistor SMD 0805 (2012 Metric), square (rectangular) end terminal, IPC_7351 nominal with elongated pad for handsoldering. (Body size source: https://docs.google.com/spreadsheets/d/1BsfQQcO9C6DZCsRaXUlFlo91Tg2WpOkGARC1WS5S8t0/edit?usp=sharing), generated with kicad-footprint-generator")
     (tags "resistor handsolder")
     (attr smd)
-    (fp_text reference R7 (at 0 -1.65) (layer F.SilkS)
+    (fp_text reference R7 (at 0 1.5) (layer F.SilkS)
       (effects (font (size 1 1) (thickness 0.15)))
     )
@@
     (tags "resistor handsolder")
     (attr smd)
-    (fp_text reference R6 (at 0 -1.65) (layer F.SilkS)
+    (fp_text reference R6 (at 0 1.5) (layer F.SilkS)
       (effects (font (size 1 1) (thickness 0.15)))
     )
@@
     (tags "resistor handsolder")
     (attr smd)
-    (fp_text reference R5 (at 0 -1.65 90) (layer F.SilkS)
+    (fp_text reference R5 (at -0.9 -1.65 90) (layer F.SilkS)
       (effects (font (size 1 1) (thickness 0.15)))
     )
@@
     (tags "resistor handsolder")
     (attr smd)
-    (fp_text reference R4 (at 0 -1.65 90) (layer F.SilkS)
+    (fp_text reference R4 (at -0.1 1.7 90) (layer F.SilkS)
       (effects (font (size 1 1) (thickness 0.15)))
     )
@@
     (tags "resistor handsolder")
     (attr smd)
-    (fp_text reference R3 (at 0 -1.65 90) (layer F.SilkS)
+    (fp_text reference R3 (at 0 7.9 90) (layer F.SilkS)
       (effects (font (size 1 1) (thickness 0.15)))
     )
@@
     (tags "resistor handsolder")
     (attr smd)
-    (fp_text reference R2 (at 0 -1.65 90) (layer F.SilkS)
+    (fp_text reference R2 (at 0 6.3 90) (layer F.SilkS)
       (effects (font (size 1 1) (thickness 0.15)))
     )
@@
     (tags "resistor handsolder")
     (attr smd)
-    (fp_text reference R1 (at 0 -1.65 90) (layer F.SilkS)
+    (fp_text reference R1 (at 0 4.6 90) (layer F.SilkS)
       (effects (font (size 1 1) (thickness 0.15)))
     )
@@
     (descr "15-pin D-Sub connector, horizontal/angled (90 deg), THT-mount, female, pitch 2.29x1.98mm, pin-PCB-offset 3.0300000000000002mm, distance of mounting holes 25mm, distance of mounting holes to PCB edge 4.9399999999999995mm, see https://disti-assets.s3.amazonaws.com/tonar/files/datasheets/16730.pdf")
     (tags "15-pin D-Sub connector horizontal angled 90deg THT female pitch 2.29x1.98mm pin-PCB-offset 3.0300000000000002mm mounting-holes-distance 25mm mounting-hole-offset 25mm")
-    (fp_text reference J2 (at -4.315 -2.61) (layer F.SilkS)
+    (fp_text reference J2 (at -21.5 5.7) (layer F.SilkS)
       (effects (font (size 1 1) (thickness 0.15)))
     )
@@
     (tags "inductor handsolder")
     (attr smd)
-    (fp_text reference FB1 (at 0 -1.65 90) (layer F.SilkS)
+    (fp_text reference FB1 (at 0 1.7 90) (layer F.SilkS)
       (effects (font (size 1 1) (thickness 0.15)))
     )
@@
   )
   (module Capacitor_SMD:C_0805_2012Metric_Pad1.15x1.40mm_HandSolder (layer F.Cu)
-    (at 0 -15 180)
+    (at 0 -12.75 180)
     (descr "Capacitor SMD 0805 (2012 Metric), square (rectangular) end terminal, IPC_7351 nominal with elongated pad for handsoldering. (Body size source: https://docs.google.com/spreadsheets/d/1BsfQQcO9C6DZCsRaXUlFlo91Tg2WpOkGARC1WS5S8t0/edit?usp=sharing), generated with kicad-footprint-generator")
     (tags "capacitor handsolder")
@@
     (tags "capacitor handsolder")
     (attr smd)
-    (fp_text reference C17 (at 0 -1.65) (layer F.SilkS)
+    (fp_text reference C17 (at 3.3 0) (layer F.SilkS)
       (effects (font (size 1 1) (thickness 0.15)))
     )
@@
     (tags "capacitor handsolder")
     (attr smd)
-    (fp_text reference C15 (at 0 -1.65 90) (layer F.SilkS)
+    (fp_text reference C15 (at 0 1.7 90) (layer F.SilkS)
       (effects (font (size 1 1) (thickness 0.15)))
     )
@@
     (tags "capacitor handsolder")
     (attr smd)
-    (fp_text reference C11 (at 0 -1.65 90) (layer F.SilkS)
+    (fp_text reference C11 (at 0 -4.1 90) (layer F.SilkS)
       (effects (font (size 1 1) (thickness 0.15)))
     )
@@
     (tags "capacitor handsolder")
     (attr smd)
-    (fp_text reference C10 (at 0 -1.65 90) (layer F.SilkS)
+    (fp_text reference C10 (at -3.5 3.2 90) (layer F.SilkS)
       (effects (font (size 1 1) (thickness 0.15)))
     )
@@
     (tags "capacitor handsolder")
     (attr smd)
-    (fp_text reference C9 (at 0 -1.65 90) (layer F.SilkS)
+    (fp_text reference C9 (at 0 3 90) (layer F.SilkS)
       (effects (font (size 1 1) (thickness 0.15)))
     )
@@
     (tags "capacitor tantalum")
     (attr smd)
-    (fp_text reference C8 (at 0 -2.35 90) (layer F.SilkS)
+    (fp_text reference C8 (at 0 2.3 90) (layer F.SilkS)
       (effects (font (size 1 1) (thickness 0.15)))
     )
@@
     (tags "capacitor handsolder")
     (attr smd)
-    (fp_text reference C7 (at 0 -1.65) (layer F.SilkS)
+    (fp_text reference C7 (at 0 1.65) (layer F.SilkS)
       (effects (font (size 1 1) (thickness 0.15)))
     )
@@
     (descr "CP, Radial series, Radial, pin pitch=3.50mm, , diameter=8mm, Electrolytic Capacitor")
     (tags "CP Radial series Radial pin pitch 3.50mm  diameter 8mm Electrolytic Capacitor")
-    (fp_text reference C3 (at 1.75 -5.25 90) (layer F.SilkS)
+    (fp_text reference C3 (at 1.7 5.2 90) (layer F.SilkS)
       (effects (font (size 1 1) (thickness 0.15)))
     )
@@
     (descr "CP, Radial series, Radial, pin pitch=3.50mm, , diameter=8mm, Electrolytic Capacitor")
     (tags "CP Radial series Radial pin pitch 3.50mm  diameter 8mm Electrolytic Capacitor")
-    (fp_text reference C2 (at 1.75 -5.25 90) (layer F.SilkS)
+    (fp_text reference C2 (at 4.6 4.7 90) (layer F.SilkS)
       (effects (font (size 1 1) (thickness 0.15)))
     )
@@
     )
   )
+  (gr_line (start 0.7 -6.4) (end 0.3 -6.4) (layer F.SilkS) (width 0.15))
+  (gr_line (start 0.3 -6.4) (end -0.2 -6.4) (layer F.SilkS) (width 0.15))
+  (gr_line (start 1 -5.2) (end 0.3 -6.4) (layer F.SilkS) (width 0.15))
+  (gr_line (start 2.6 -5.2) (end 1 -5.2) (layer F.SilkS) (width 0.15))
+  (gr_line (start 2.6 -5.6) (end 2.6 -4.9) (layer F.SilkS) (width 0.15))
+  (gr_line (start 24 -11.5) (end 18 -11.5) (layer B.SilkS) (width 0.15))
+  (gr_line (start 24 -27.5) (end 24 -11.5) (layer B.SilkS) (width 0.15))
+  (gr_line (start 18 -27.5) (end 24 -27.5) (layer B.SilkS) (width 0.15))
+  (gr_line (start 18 -11.5) (end 18 -27.5) (layer B.SilkS) (width 0.15))
+  (gr_text "Nuno Sousa\n10/2020" (at 21 -19.5 90) (layer B.SilkS)
+    (effects (font (size 1.5 1.5) (thickness 0.3)) (justify mirror))
+  )
   (gr_circle (center 14 -14) (end 17.3 -14) (layer Dwgs.User) (width 0.1))
   (gr_circle (center -14 -14) (end -10.7 -14) (layer Dwgs.User) (width 0.1))
@@
   (segment (start -23 8.75) (end -22.75 8.5) (width 0.4) (layer F.Cu) (net 7))
   (segment (start -23 10.67) (end -23 8.75) (width 0.4) (layer F.Cu) (net 7))
+  (via (at -18.75 2.75) (size 0.8) (drill 0.4) (layers F.Cu B.Cu) (net 7))
   (segment (start -2.00001 -8.52499) (end -1 -9.525) (width 0.35) (layer F.Cu) (net 8))
   (segment (start -5.49999 -8.52499) (end -2.00001 -8.52499) (width 0.35) (layer F.Cu) (net 8))
@@
   (segment (start -23.65 10.67) (end -23.65 8.25) (width 0.4) (layer F.Cu) (net 33))
   (zone (net 7) (net_name GND) (layer F.Cu) (hatch edge 0.508)
-    (connect_pads (clearance 0.508))
+    (connect_pads (clearance 0.254))
     (min_thickness 0.254)
     (fill yes (arc_segments 32) (thermal_gap 0.508) (thermal_bridge_width 0.508) (smoothing fillet) (radius 1))
@@
   )
   (zone (net 7) (net_name GND) (layer B.Cu) (hatch edge 0.508)
-    (connect_pads (clearance 0.508))
+    (connect_pads (clearance 0.254))
     (min_thickness 0.254)
     (fill yes (arc_segments 32) (thermal_gap 0.508) (thermal_bridge_width 0.508) (smoothing fillet) (radius 1))
