File: Hardware/Dreamcast_VGA_Adapter.kicad_pcb (KiCad board)
At the start: 2 copper layers, 56.6 x 57.7 mm, 41 parts, among them J1 AudioJack3, J2 DB15_Female_HighDensity_Mount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, J3 Conn_02x08_Odd_Even, SW1 SW_DIP_x02, U1 THS7316, U2 74HCT2G34

Commit message: Updated 3D design.
Parts:
- moved J1 1.00 mm to (23.0, 26.5)
Routing:
- net /AUDIO-R: track 52.6 -> 51.6 mm, vias 1 -> 0

Commit message: Updated PCB.
Parts:
- moved J1 0.50 mm to (22.5, 26.5)
Routing:
- net /H-SYNC: track 53.4 -> 55.5 mm
- net /AUDIO-L: track 57.0 -> 59.0 mm
- net /V-SYNC: track 45.8 -> 47.6 mm
- net /AUDIO-R: track 51.6 -> 52.1 mm
- net GND: vias 77 -> 80
Other:
- board text added: "15kHz RGB (SCART)"
- board text added: "31kHz RGB (VGA)"
- board text added: "Standard 'TV'"
Changed lines of the file:
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@@
   (general
     (thickness 1.6)
-    (drawings 30)
-    (tracks 325)
+    (drawings 64)
+    (tracks 340)
     (zones 0)
     (modules 41)
@@
     (46 B.CrtYd user)
     (47 F.CrtYd user)
-    (48 B.Fab user hide)
-    (49 F.Fab user)
+    (48 B.Fab user)
+    (49 F.Fab user hide)
   )
   (setup
@@
   )
   (module Connector_Audio_custom:Jack_3.5mm_CUI_SJ1-3533NG_Horizontal (layer F.Cu)
-    (at 23 26.5 180)
+    (at 22.5 26.5 180)
     (descr "TRS 3.5mm, horizontal, through-hole, https://www.cui.com/product/resource/sj1-353xng.pdf")
     (tags "TRS audio jack stereo horizontal")
@@
     )
   )
+  (gr_text "Standard\n'TV'" (at 20.25 10.5) (layer F.SilkS)
+    (effects (font (size 1 1) (thickness 0.15)))
+  )
+  (gr_line (start 18.365 4.41) (end 19.635 4.41) (layer F.SilkS) (width 0.15))
+  (gr_line (start 19.635 4.41) (end 19.635 8.47) (layer F.SilkS) (width 0.15))
+  (gr_line (start 22.175 8.47) (end 20.905 8.47) (layer F.SilkS) (width 0.15))
+  (gr_line (start 19.635 8.47) (end 18.365 8.47) (layer F.SilkS) (width 0.15))
+  (gr_poly (pts (xy 19.635 5.75) (xy 18.365 5.75) (xy 18.365 4.396667) (xy 19.635 4.396667)) (layer F.SilkS) (width 0.1))
+  (gr_line (start 22.175 4.41) (end 22.175 8.47) (layer F.SilkS) (width 0.15))
+  (gr_poly (pts (xy 22.175 5.763333) (xy 20.905 5.763333) (xy 20.905 4.41) (xy 22.175 4.41)) (layer F.SilkS) (width 0.1))
+  (gr_line (start 18.365 8.47) (end 18.365 4.41) (layer F.SilkS) (width 0.15))
+  (gr_line (start 20.905 4.41) (end 22.175 4.41) (layer F.SilkS) (width 0.15))
+  (gr_line (start 20.905 8.47) (end 20.905 4.41) (layer F.SilkS) (width 0.15))
+  (gr_text "15kHz\nRGB (SCART)" (at 20.5 1.75) (layer F.SilkS)
+    (effects (font (size 1 1) (thickness 0.15)))
+  )
+  (gr_line (start 22.425 -4.34) (end 22.425 -0.28) (layer F.SilkS) (width 0.15))
+  (gr_line (start 18.615 -0.28) (end 18.615 -4.34) (layer F.SilkS) (width 0.15))
+  (gr_line (start 21.155 -0.28) (end 21.155 -4.34) (layer F.SilkS) (width 0.15))
+  (gr_line (start 21.155 -4.34) (end 22.425 -4.34) (layer F.SilkS) (width 0.15))
+  (gr_poly (pts (xy 22.425 -0.28) (xy 21.155 -0.28) (xy 21.155 -1.633333) (xy 22.425 -1.633333)) (layer F.SilkS) (width 0.1))
+  (gr_line (start 22.425 -0.28) (end 21.155 -0.28) (layer F.SilkS) (width 0.15))
+  (gr_line (start 18.615 -4.34) (end 19.885 -4.34) (layer F.SilkS) (width 0.15))
+  (gr_line (start 19.885 -4.34) (end 19.885 -0.28) (layer F.SilkS) (width 0.15))
+  (gr_line (start 19.885 -0.28) (end 18.615 -0.28) (layer F.SilkS) (width 0.15))
+  (gr_poly (pts (xy 19.885 -3) (xy 18.615 -3) (xy 18.615 -4.353333) (xy 19.885 -4.353333)) (layer F.SilkS) (width 0.1))
+  (gr_text "31kHz\nRGB (VGA)" (at 20.55 -20.15) (layer F.SilkS)
+    (effects (font (size 1 1) (thickness 0.15)))
+  )
+  (gr_line (start -22 -16) (end -22.5 -16) (layer F.SilkS) (width 0.15))
+  (gr_poly (pts (xy 19.935 -22.18) (xy 18.665 -22.18) (xy 18.665 -23.533333) (xy 19.935 -23.533333)) (layer F.SilkS) (width 0.1))
+  (gr_poly (pts (xy 22.475 -22.18) (xy 21.205 -22.18) (xy 21.205 -23.533333) (xy 22.475 -23.533333)) (layer F.SilkS) (width 0.1))
+  (gr_line (start 21.205 -22.18) (end 21.205 -26.24) (layer F.SilkS) (width 0.15))
+  (gr_line (start 22.475 -22.18) (end 21.205 -22.18) (layer F.SilkS) (width 0.15))
+  (gr_line (start 22.475 -26.24) (end 22.475 -22.18) (layer F.SilkS) (width 0.15))
+  (gr_line (start 21.205 -26.24) (end 22.475 -26.24) (layer F.SilkS) (width 0.15))
+  (gr_line (start 18.665 -22.18) (end 18.665 -26.24) (layer F.SilkS) (width 0.15))
+  (gr_line (start 19.935 -22.18) (end 18.665 -22.18) (layer F.SilkS) (width 0.15))
+  (gr_line (start 19.935 -26.24) (end 19.935 -22.18) (layer F.SilkS) (width 0.15))
+  (gr_line (start 18.665 -26.24) (end 19.935 -26.24) (layer F.SilkS) (width 0.15))
   (gr_line (start 0.7 -6.4) (end 0.3 -6.4) (layer F.SilkS) (width 0.15))
   (gr_line (start 0.3 -6.4) (end -0.2 -6.4) (layer F.SilkS) (width 0.15))
@@
   (via (at 25 25) (size 0.8) (drill 0.4) (layers F.Cu B.Cu) (net 7))
   (via (at -10 -15) (size 0.8) (drill 0.4) (layers F.Cu B.Cu) (net 7))
+  (via (at 3 -6.75) (size 0.8) (drill 0.4) (layers F.Cu B.Cu) (net 7))
+  (via (at -2.5 -7) (size 0.8) (drill 0.4) (layers F.Cu B.Cu) (net 7))
+  (via (at 7.5 -4.5) (size 0.8) (drill 0.4) (layers F.Cu B.Cu) (net 7))
   (segment (start -2.00001 -8.52499) (end -1 -9.525) (width 0.35) (layer F.Cu) (net 8))
   (segment (start -5.49999 -8.52499) (end -2.00001 -8.52499) (width 0.35) (layer F.Cu) (net 8))
@@
   (segment (start 9.5 -15.57) (end 9.5 -12.025) (width 1) (layer F.Cu) (net 15))
   (segment (start 3.81 -21.26) (end 9.5 -15.57) (width 1) (layer F.Cu) (net 15))
-  (segment (start 22.3 17.3) (end 21 18.6) (width 1) (layer F.Cu) (net 16))
   (segment (start 20 -4.05) (end 22.3 -1.75) (width 1) (layer F.Cu) (net 16))
   (segment (start 20 -10.25) (end 20 -4.05) (width 1) (layer F.Cu) (net 16))
@@
   (segment (start 16.94 -21.26) (end 21.150001 -17.049999) (width 1) (layer F.Cu) (net 16))
   (segment (start 8.89 -21.26) (end 16.94 -21.26) (width 1) (layer F.Cu) (net 16))
+  (segment (start 21 18.6) (end 22.3 17.3) (width 1) (layer F.Cu) (net 16))
+  (segment (start 20.5 18.6) (end 21 18.6) (width 1) (layer F.Cu) (net 16))
   (segment (start 20 24.1) (end 21 24.1) (width 1) (layer F.Cu) (net 17))
-  (segment (start 18.4 22.5) (end 20 24.1) (width 1) (layer F.Cu) (net 17))
-  (segment (start 18.4 10.7) (end 18.4 22.5) (width 1) (layer F.Cu) (net 17))
   (segment (start 17.1 9.4) (end 18.4 10.7) (width 1) (layer F.Cu) (net 17))
   (segment (start 17.1 -10.6) (end 17.1 9.4) (width 1) (layer F.Cu) (net 17))
@@
   (segment (start 18.3 -16.2) (end 18.3 -11.8) (width 1) (layer F.Cu) (net 17))
   (segment (start 6.35 -21.26) (end 9.11 -18.5) (width 1) (layer F.Cu) (net 17))
+  (segment (start 20.5 24.1) (end 19.5 24.1) (width 1) (layer F.Cu) (net 17))
+  (segment (start 19.5 24.1) (end 17 21.6) (width 1) (layer F.Cu) (net 17))
+  (segment (start 17 21.6) (end 17 17.45) (width 1) (layer F.Cu) (net 17))
+  (segment (start 18.4 16.05) (end 18.4 10.7) (width 1) (layer F.Cu) (net 17))
+  (segment (start 17 17.45) (end 18.4 16.05) (width 1) (layer F.Cu) (net 17))
   (segment (start -21.025 17.5) (end -21.025 15.975) (width 0.5) (layer F.Cu) (net 19))
   (segment (start -21.025 15.975) (end -22 15) (width 0.5) (layer F.Cu) (net 19))
@@
   (segment (start 0 -22.53) (end 0 -22.8) (width 0.5) (layer F.Cu) (net 28))
   (segment (start 0 -22.8) (end 0 -24.7) (width 0.25) (layer F.Cu) (net 28))
-  (segment (start -21.7 2.6) (end -23.5 4.4) (width 0.5) (layer F.Cu) (net 28))
-  (segment (start -20.35 2.6) (end -21.7 2.6) (width 0.5) (layer F.Cu) (net 28))
-  (segment (start -23.5 4.4) (end -23.5 4.975) (width 0.5) (layer F.Cu) (net 28))
-  (segment (start -18.3 0.55) (end -20.35 2.6) (width 0.5) (layer F.Cu) (net 28))
-  (segment (start -18.3 -19.8) (end -18.3 0.55) (width 0.5) (layer F.Cu) (net 28))
-  (segment (start -1.3 -26.2) (end -11.9 -26.2) (width 0.5) (layer F.Cu) (net 28))
-  (segment (start -11.9 -26.2) (end -18.3 -19.8) (width 0.5) (layer F.Cu) (net 28))
-  (segment (start 0 -24.9) (end -1.3 -26.2) (width 0.5) (layer F.Cu) (net 28))
-  (segment (start 0 -24.7) (end 0 -24.9) (width 0.5) (layer F.Cu) (net 28))
+  (segment (start 0 -24.9) (end 0 -24.7) (width 0.5) (layer F.Cu) (net 28))
+  (segment (start -1.3 -26.2) (end 0 -24.9) (width 0.5) (layer F.Cu) (net 28))
+  (segment (start -18.3 -18.032002) (end -18.3 -19.8) (width 0.5) (layer F.Cu) (net 28))
+  (segment (start -20.900001 -15.432001) (end -18.3 -18.032002) (width 0.5) (layer F.Cu) (net 28))
+  (segment (start -11.9 -26.2) (end -1.3 -26.2) (width 0.5) (layer F.Cu) (net 28))
+  (segment (start -18.3 0.55) (end -18.3 -9.7) (width 0.5) (layer F.Cu) (net 28))
+  (segment (start -18.3 -19.8) (end -11.9 -26.2) (width 0.5) (layer F.Cu) (net 28))
+  (segment (start -20.900001 -12.300001) (end -20.900001 -15.432001) (width 0.5) (layer F.Cu) (net 28))
+  (segment (start -20.35 2.6) (end -18.3 0.55) (width 0.5) (layer F.Cu) (net 28))
+  (segment (start -21.7 2.6) (end -20.35 2.6) (width 0.5) (layer F.Cu) (net 28))
+  (segment (start -23.5 4.4) (end -21.7 2.6) (width 0.5) (layer F.Cu) (net 28))
+  (segment (start -18.3 -9.7) (end -20.900001 -12.300001) (width 0.5) (layer F.Cu) (net 28))
+  (segment (start -23.5 4.975) (end -23.5 4.4) (width 0.5) (layer F.Cu) (net 28))
   (segment (start -1.27 -24.47) (end -1.27 -23.8) (width 0.5) (layer F.Cu) (net 29))
+  (segment (start -2.2 -25.4) (end -1.27 -24.47) (width 0.5) (layer F.Cu) (net 29))
   (segment (start -10 -25.4) (end -2.2 -25.4) (width 0.5) (layer F.Cu) (net 29))
+  (segment (start -16.6 -18.8) (end -10 -25.4) (width 0.5) (layer F.Cu) (net 29))
+  (segment (start -18.75 -15.4) (end -16.6 -17.55) (width 0.5) (layer F.Cu) (net 29))
+  (segment (start -18.75 -12.55) (end -18.75 -15.4) (width 0.5) (layer F.Cu) (net 29))
+  (segment (start -16.6 -10.4) (end -18.75 -12.55) (width 0.5) (layer F.Cu) (net 29))
+  (segment (start -16.6 -17.55) (end -16.6 -18.8) (width 0.5) (layer F.Cu) (net 29))
+  (segment (start -16.6 2.4) (end -16.6 -10.4) (width 0.5) (layer F.Cu) (net 29))
+  (segment (start -19.175 4.975) (end -16.6 2.4) (width 0.5) (layer F.Cu) (net 29))
   (segment (start -21 4.975) (end -19.175 4.975) (width 0.5) (layer F.Cu) (net 29))
-  (segment (start -19.175 4.975) (end -16.6 2.4) (width 0.5) (layer F.Cu) (net 29))
-  (segment (start -16.6 2.4) (end -16.6 -18.8) (width 0.5) (layer F.Cu) (net 29))
-  (segment (start -2.2 -25.4) (end -1.27 -24.47) (width 0.5) (layer F.Cu) (net 29))
-  (segment (start -16.6 -18.8) (end -10 -25.4) (width 0.5) (layer F.Cu) (net 29))
   (segment (start 2.571399 -23.071399) (end 2.571399 -24.628601) (width 0.25) (layer F.Cu) (net 30))
   (segment (start 2.571399 -22.561399) (end 2.571399 -23.071399) (width 0.5) (layer F.Cu) (net 30))

Commit message: Upgraded from Kicad 5 to Kicad 8.
Other:
- net class 75ohm_track removed
- net class Default removed
- net class Power removed
